Commit message: added new urdf

File: hexapod_control/ros2_control/ros2_control.xacro (robot description, xacro)
@@ -6,243 +6,243 @@
     <plugin>ign_ros2_control/IgnitionSystem</plugin>
   </hardware>
-  <joint name="Revolute_63">
-    <command_interface name="position">
-    <param name="min">-1.57</param>
-    <param name="max">1.57</param>
-    </command_interface>
-    <state_interface name="position">
-        <param name="initial_value">0</param>
-    </state_interface>
-    <state_interface name="velocity"/>
-    <state_interface name="effort"/>
-    <limit>
-      <velocity>100.0</velocity>
-    </limit>
-  </joint>
-  <joint name="Revolute_64">
-    <command_interface name="position">
-    <param name="min">-1.57</param>
-    <param name="max">1.57</param>
-    </command_interface>
-    <state_interface name="position">
-        <param name="initial_value">0</param>
-    </state_interface>
-    <state_interface name="velocity"/>
-    <state_interface name="effort"/>
-    <limit>
-      <velocity>100.0</velocity>
-    </limit>
-  </joint>
-  <joint name="Revolute_65">
-    <command_interface name="position">
-    <param name="min">-1.57</param>
-    <param name="max">1.57</param>
-    </command_interface>
-    <state_interface name="position">
-        <param name="initial_value">0</param>
-    </state_interface>
-    <state_interface name="velocity"/>
-    <state_interface name="effort"/>
-    <limit>
-      <velocity>100.0</velocity>
-    </limit>
-  </joint>
-  <joint name="Revolute_69">
-    <command_interface name="position">
-    <param name="min">-1.57</param>
-    <param name="max">1.57</param>
-    </command_interface>
-    <state_interface name="position">
-        <param name="initial_value">0</param>
-    </state_interface>
-    <state_interface name="velocity"/>
-    <state_interface name="effort"/>
-    <limit>
-      <velocity>100.0</velocity>
-    </limit>
-  </joint>
-  <joint name="Revolute_70">
-    <command_interface name="position">
-    <param name="min">-1.57</param>
-    <param name="max">1.57</param>
-    </command_interface>
-    <state_interface name="position">
-        <param name="initial_value">0</param>
-    </state_interface>
-    <state_interface name="velocity"/>
-    <state_interface name="effort"/>
-    <limit>
-      <velocity>100.0</velocity>
-    </limit>
-  </joint>
-  <joint name="Revolute_71">
-    <command_interface name="position">
-    <param name="min">-1.57</param>
-    <param name="max">1.57</param>
-    </command_interface>
-    <state_interface name="position">
-        <param name="initial_value">0</param>
-    </state_interface>
-    <state_interface name="velocity"/>
-    <state_interface name="effort"/>
-    <limit>
-      <velocity>100.0</velocity>
-    </limit>
-  </joint>
-  <joint name="Revolute_72">
-    <command_interface name="position">
-    <param name="min">-1.57</param>
-    <param name="max">1.57</param>
-    </command_interface>
-    <state_interface name="position">
-        <param name="initial_value">0</param>
-    </state_interface>
-    <state_interface name="velocity"/>
-    <state_interface name="effort"/>
-    <limit>
-      <velocity>100.0</velocity>
-    </limit>
-  </joint>
-  <joint name="Revolute_73">
-    <command_interface name="position">
-    <param name="min">-1.57</param>
-    <param name="max">1.57</param>
-    </command_interface>
-    <state_interface name="position">
-        <param name="initial_value">0</param>
-    </state_interface>
-    <state_interface name="velocity"/>
-    <state_interface name="effort"/>
-    <limit>
-      <velocity>100.0</velocity>
-    </limit>
-  </joint>
-  <joint name="Revolute_74">
-    <command_interface name="position">
-    <param name="min">-1.57</param>
-    <param name="max">1.57</param>
-    </command_interface>
-    <state_interface name="position">
-        <param name="initial_value">0</param>
-    </state_interface>
-    <state_interface name="velocity"/>
-    <state_interface name="effort"/>
-    <limit>
-      <velocity>100.0</velocity>
-    </limit>
-  </joint>
-  <joint name="Revolute_75">
-    <command_interface name="position">
-    <param name="min">-1.57</param>
-    <param name="max">1.57</param>
-    </command_interface>
-    <state_interface name="position">
-        <param name="initial_value">0</param>
-    </state_interface>
-    <state_interface name="velocity"/>
-    <state_interface name="effort"/>
-    <limit>
-      <velocity>100.0</velocity>
-    </limit>
-  </joint>
-  <joint name="Revolute_76">
-    <command_interface name="position">
-    <param name="min">-1.57</param>
-    <param name="max">1.57</param>
-    </command_interface>
-    <state_interface name="position">
-        <param name="initial_value">0</param>
-    </state_interface>
-    <state_interface name="velocity"/>
-    <state_interface name="effort"/>
-    <limit>
-      <velocity>100.0</velocity>
-    </limit>
-  </joint>
-  <joint name="Revolute_77">
-    <command_interface name="position">
-    <param name="min">-1.57</param>
-    <param name="max">1.57</param>
-    </command_interface>
-    <state_interface name="position">
-        <param name="initial_value">0</param>
-    </state_interface>
-    <state_interface name="velocity"/>
-    <state_interface name="effort"/>
-    <limit>
-      <velocity>100.0</velocity>
-    </limit>
-  </joint>
-  <joint name="Revolute_78">
-    <command_interface name="position">
-    <param name="min">-1.57</param>
-    <param name="max">1.57</param>
-    </command_interface>
-    <state_interface name="position">
-        <param name="initial_value">0</param>
-    </state_interface>
-    <state_interface name="velocity"/>
-    <state_interface name="effort"/>
-    <limit>
-      <velocity>100.0</velocity>
-    </limit>
-  </joint>
-  <joint name="Revolute_79">
-    <command_interface name="position">
-    <param name="min">-1.57</param>
-    <param name="max">1.57</param>
-    </command_interface>
-    <state_interface name="position">
-        <param name="initial_value">0</param>
-    </state_interface>
-    <state_interface name="velocity"/>
-    <state_interface name="effort"/>
-    <limit>
-      <velocity>100.0</velocity>
-    </limit>
-  </joint>
-  <joint name="Revolute_80">
-    <command_interface name="position">
-    <param name="min">-1.57</param>
-    <param name="max">1.57</param>
-    </command_interface>
-    <state_interface name="position">
-        <param name="initial_value">0</param>
-    </state_interface>
-    <state_interface name="velocity"/>
-    <state_interface name="effort"/>
-    <limit>
-      <velocity>100.0</velocity>
-    </limit>
-  </joint>
-  <joint name="Revolute_81">
-    <command_interface name="position">
-    <param name="min">-1.57</param>
-    <param name="max">1.57</param>
-    </command_interface>
-    <state_interface name="position">
-        <param name="initial_value">0</param>
-    </state_interface>
-    <state_interface name="velocity"/>
-    <state_interface name="effort"/>
-    <limit>
-      <velocity>100.0</velocity>
-    </limit>
-  </joint>
-  <joint name="Revolute_82">
-    <command_interface name="position">
-    <param name="min">-1.57</param>
-    <param name="max">1.57</param>
-    </command_interface>
-    <state_interface name="position">
-        <param name="initial_value">0</param>
-    </state_interface>
-    <state_interface name="velocity"/>
-    <state_interface name="effort"/>
-    <limit>
-      <velocity>100.0</velocity>
-    </limit>
-  </joint>
-  <joint name="Revolute_83">
+  <joint name="Leg_1_coxa">
+    <command_interface name="position">
+    <param name="min">-1.57</param>
+    <param name="max">1.57</param>
+    </command_interface>
+    <state_interface name="position">
+        <param name="initial_value">0</param>
+    </state_interface>
+    <state_interface name="velocity"/>
+    <state_interface name="effort"/>
+    <limit>
+      <velocity>100.0</velocity>
+    </limit>
+  </joint>
+  <joint name="Leg_2_coxa">
+    <command_interface name="position">
+    <param name="min">-1.57</param>
+    <param name="max">1.57</param>
+    </command_interface>
+    <state_interface name="position">
+        <param name="initial_value">0</param>
+    </state_interface>
+    <state_interface name="velocity"/>
+    <state_interface name="effort"/>
+    <limit>
+      <velocity>100.0</velocity>
+    </limit>
+  </joint>
+  <joint name="Leg_3_coxa">
+    <command_interface name="position">
+    <param name="min">-1.57</param>
+    <param name="max">1.57</param>
+    </command_interface>
+    <state_interface name="position">
+        <param name="initial_value">0</param>
+    </state_interface>
+    <state_interface name="velocity"/>
+    <state_interface name="effort"/>
+    <limit>
+      <velocity>100.0</velocity>
+    </limit>
+  </joint>
+  <joint name="Leg_1_tibia">
+    <command_interface name="position">
+    <param name="min">-1.57</param>
+    <param name="max">1.57</param>
+    </command_interface>
+    <state_interface name="position">
+        <param name="initial_value">0</param>
+    </state_interface>
+    <state_interface name="velocity"/>
+    <state_interface name="effort"/>
+    <limit>
+      <velocity>100.0</velocity>
+    </limit>
+  </joint>
+  <joint name="Leg_2_tibia">
+    <command_interface name="position">
+    <param name="min">-1.57</param>
+    <param name="max">1.57</param>
+    </command_interface>
+    <state_interface name="position">
+        <param name="initial_value">0</param>
+    </state_interface>
+    <state_interface name="velocity"/>
+    <state_interface name="effort"/>
+    <limit>
+      <velocity>100.0</velocity>
+    </limit>
+  </joint>
+  <joint name="Leg_3_tibia">
+    <command_interface name="position">
+    <param name="min">-1.57</param>
+    <param name="max">1.57</param>
+    </command_interface>
+    <state_interface name="position">
+        <param name="initial_value">0</param>
+    </state_interface>
+    <state_interface name="velocity"/>
+    <state_interface name="effort"/>
+    <limit>
+      <velocity>100.0</velocity>
+    </limit>
+  </joint>
+  <joint name="Leg_1_femur">
+    <command_interface name="position">
+    <param name="min">-1.57</param>
+    <param name="max">1.57</param>
+    </command_interface>
+    <state_interface name="position">
+        <param name="initial_value">0</param>
+    </state_interface>
+    <state_interface name="velocity"/>
+    <state_interface name="effort"/>
+    <limit>
+      <velocity>100.0</velocity>
+    </limit>
+  </joint>
+  <joint name="Leg_2_femur">
+    <command_interface name="position">
+    <param name="min">-1.57</param>
+    <param name="max">1.57</param>
+    </command_interface>
+    <state_interface name="position">
+        <param name="initial_value">0</param>
+    </state_interface>
+    <state_interface name="velocity"/>
+    <state_interface name="effort"/>
+    <limit>
+      <velocity>100.0</velocity>
+    </limit>
+  </joint>
+  <joint name="Leg_3_femur">
+    <command_interface name="position">
+    <param name="min">-1.57</param>
+    <param name="max">1.57</param>
+    </command_interface>
+    <state_interface name="position">
+        <param name="initial_value">0</param>
+    </state_interface>
+    <state_interface name="velocity"/>
+    <state_interface name="effort"/>
+    <limit>
+      <velocity>100.0</velocity>
+    </limit>
+  </joint>
+  <joint name="Leg_6_femur">
+    <command_interface name="position">
+    <param name="min">-1.57</param>
+    <param name="max">1.57</param>
+    </command_interface>
+    <state_interface name="position">
+        <param name="initial_value">0</param>
+    </state_interface>
+    <state_interface name="velocity"/>
+    <state_interface name="effort"/>
+    <limit>
+      <velocity>100.0</velocity>
+    </limit>
+  </joint>
+  <joint name="Leg_4_coxa">
+    <command_interface name="position">
+    <param name="min">-1.57</param>
+    <param name="max">1.57</param>
+    </command_interface>
+    <state_interface name="position">
+        <param name="initial_value">0</param>
+    </state_interface>
+    <state_interface name="velocity"/>
+    <state_interface name="effort"/>
+    <limit>
+      <velocity>100.0</velocity>
+    </limit>
+  </joint>
+  <joint name="Leg_5_coxa">
+    <command_interface name="position">
+    <param name="min">-1.57</param>
+    <param name="max">1.57</param>
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