Commit message: joint position control

File: hexapod_description/urdf/hexapod.xacro (robot description, xacro)
@@ -7,7 +7,7 @@
 <link name="base_link">
   <inertial>
-    <origin xyz="0.1000352418955988 0.06495559041692857 0.006960329203092366" rpy="0 0 0"/>
+    <origin xyz="0.10909777793044037 0.06468612005136756 0.006889314215312581" rpy="0 0 0"/>
     <mass value="14.09466584247892"/>
-    <inertia ixx="0.167546" iyy="0.075339" izz="0.199615" ixy="-0.012339" iyz="0.003184" ixz="-0.003868"/>
+    <inertia ixx="0.168182" iyy="0.074083" izz="0.200235" ixy="0.006215" iyz="0.001309" ixz="-0.000356"/>
   </inertial>
   <visual>
@@ -27,10 +27,10 @@
 <link name="leg_1_link_2_1">
   <inertial>
-    <origin xyz="-0.020798247907869903 -0.003004122621169035 -0.05840364105605461" rpy="0 0 0"/>
+    <origin xyz="-0.02800590467788834 0.004191461427254562 -0.05523214859518318" rpy="0 0 0"/>
     <mass value="1.012661950148346"/>
-    <inertia ixx="0.001014" iyy="0.001236" izz="0.000891" ixy="-0.000197" iyz="-0.00022" ixz="-0.000489"/>
-  </inertial>
-  <visual>
-    <origin xyz="0.031628 0.00646 -0.021757" rpy="0 0 0"/>
+    <inertia ixx="0.000816" iyy="0.001315" izz="0.00101" ixy="-0.000122" iyz="-8.3e-05" ixz="-0.000522"/>
+  </inertial>
+  <visual>
+    <origin xyz="0.003565 0.030766 -0.036053" rpy="0 0 0"/>
     <geometry>
       <mesh filename="file://$(find hexapod_description)/meshes/leg_1_link_2_1.stl" scale="0.001 0.001 0.001"/>
@@ -39,5 +39,5 @@
   </visual>
   <collision>
-    <origin xyz="0.031628 0.00646 -0.021757" rpy="0 0 0"/>
+    <origin xyz="0.003565 0.030766 -0.036053" rpy="0 0 0"/>
     <geometry>
       <mesh filename="file://$(find hexapod_description)/meshes/leg_1_link_2_1.stl" scale="0.001 0.001 0.001"/>
@@ -47,10 +47,10 @@
 <link name="leg_1_link_3_1">
   <inertial>
-    <origin xyz="-0.05232794213563882 0.015850438170881664 0.012387465467738626" rpy="0 0 0"/>
+    <origin xyz="-0.036766491881322055 0.024823115706118865 0.034277514263341684" rpy="0 0 0"/>
     <mass value="0.22871600239093776"/>
-    <inertia ixx="0.000208" iyy="0.000275" izz="0.000422" ixy="-1e-05" iyz="1.8e-05" ixz="6.7e-05"/>
-  </inertial>
-  <visual>
-    <origin xyz="0.080903 0.053284 0.063455" rpy="0 0 0"/>
+    <inertia ixx="0.000307" iyy="0.000276" izz="0.000321" ixy="-2e-06" iyz="-2e-06" ixz="0.000128"/>
+  </inertial>
+  <visual>
+    <origin xyz="0.071402 0.062467 0.04316" rpy="0 0 0"/>
     <geometry>
       <mesh filename="file://$(find hexapod_description)/meshes/leg_1_link_3_1.stl" scale="0.001 0.001 0.001"/>
@@ -59,5 +59,5 @@
   </visual>
   <collision>
-    <origin xyz="0.080903 0.053284 0.063455" rpy="0 0 0"/>
+    <origin xyz="0.071402 0.062467 0.04316" rpy="0 0 0"/>
     <geometry>
       <mesh filename="file://$(find hexapod_description)/meshes/leg_1_link_3_1.stl" scale="0.001 0.001 0.001"/>
@@ -67,10 +67,10 @@
 <link name="leg_1_link_1_1">
   <inertial>
-    <origin xyz="-0.024118708207036738 0.023198280722906535 -0.02416394528421939" rpy="0 0 0"/>
+    <origin xyz="-0.01779410893760297 0.028725816249512953 -0.02370507712814386" rpy="0 0 0"/>
     <mass value="0.907399585528797"/>
-    <inertia ixx="0.0028" iyy="0.003123" izz="0.0006" ixy="-0.00015" iyz="-0.00034" ixz="-0.000941"/>
-  </inertial>
-  <visual>
-    <origin xyz="0.175395 0.070243 0.035462" rpy="0 0 0"/>
+    <inertia ixx="0.002849" iyy="0.003176" izz="0.000497" ixy="-2.4e-05" iyz="-1.8e-05" ixz="-0.000878"/>
+  </inertial>
+  <visual>
+    <origin xyz="0.144088 0.062627 -0.025519" rpy="0 0 0"/>
     <geometry>
       <mesh filename="file://$(find hexapod_description)/meshes/leg_1_link_1_1.stl" scale="0.001 0.001 0.001"/>
@@ -79,5 +79,5 @@
   </visual>
   <collision>
-    <origin xyz="0.175395 0.070243 0.035462" rpy="0 0 0"/>
+    <origin xyz="0.144088 0.062627 -0.025519" rpy="0 0 0"/>
     <geometry>
       <mesh filename="file://$(find hexapod_description)/meshes/leg_1_link_1_1.stl" scale="0.001 0.001 0.001"/>
@@ -87,10 +87,10 @@
 <link name="leg_3_link_3_1">
   <inertial>
-    <origin xyz="-0.01471532830032863 0.017066498243044487 -0.05783367655412228" rpy="0 0 0"/>
+    <origin xyz="-0.02800203130695705 0.004225621248029748 -0.05523202595087612" rpy="0 0 0"/>
     <mass value="1.0126620006859057"/>
-    <inertia ixx="0.000964" iyy="0.001294" izz="0.000883" ixy="0.000135" iyz="0.000218" ixz="-0.000494"/>
-  </inertial>
-  <visual>
-    <origin xyz="-0.02145 -0.24803 -0.025922" rpy="0 0 0"/>
+    <inertia ixx="0.000815" iyy="0.001315" izz="0.001011" ixy="-0.000122" iyz="-8.2e-05" ixz="-0.000522"/>
+  </inertial>
+  <visual>
+    <origin xyz="-0.00013 -0.229172 -0.040385" rpy="0 0 0"/>
     <geometry>
       <mesh filename="file://$(find hexapod_description)/meshes/leg_3_link_3_1.stl" scale="0.001 0.001 0.001"/>
@@ -99,5 +99,5 @@
   </visual>
   <collision>
-    <origin xyz="-0.02145 -0.24803 -0.025922" rpy="0 0 0"/>
+    <origin xyz="-0.00013 -0.229172 -0.040385" rpy="0 0 0"/>
     <geometry>
       <mesh filename="file://$(find hexapod_description)/meshes/leg_3_link_3_1.stl" scale="0.001 0.001 0.001"/>
@@ -107,10 +107,10 @@
 <link name="leg_3_link_2_1">
   <inertial>
-    <origin xyz="-0.02490321172110873 0.04393892851157011 0.024331856966839732" rpy="0 0 0"/>
+    <origin xyz="-0.038612908125580755 0.024931950622849613 0.03209860064693253" rpy="0 0 0"/>
     <mass value="0.2287158182027981"/>
-    <inertia ixx="0.000248" iyy="0.000272" izz="0.000385" ixy="1.3e-05" iyz="-6.3e-05" ixz="8.6e-05"/>
-  </inertial>
-  <visual>
-    <origin xyz="0.042897 -0.255314 0.061759" rpy="0 0 0"/>
+    <inertia ixx="0.000293" iyy="0.000276" izz="0.000335" ixy="-2e-06" iyz="-3e-06" ixz="0.000126"/>
+  </inertial>
+  <visual>
+    <origin xyz="0.067748 -0.197555 0.038827" rpy="0 0 0"/>
     <geometry>
       <mesh filename="file://$(find hexapod_description)/meshes/leg_3_link_2_1.stl" scale="0.001 0.001 0.001"/>
@@ -119,5 +119,5 @@
   </visual>
   <collision>
-    <origin xyz="0.042897 -0.255314 0.061759" rpy="0 0 0"/>
+    <origin xyz="0.067748 -0.197555 0.038827" rpy="0 0 0"/>
     <geometry>
       <mesh filename="file://$(find hexapod_description)/meshes/leg_3_link_2_1.stl" scale="0.001 0.001 0.001"/>
@@ -127,10 +127,10 @@
 <link name="leg_3_link_1_1">
   <inertial>
-    <origin xyz="0.008717952333481188 0.029799584273488944 -0.027197642277439673" rpy="0 0 0"/>
+    <origin xyz="-0.018585545303067386 0.028750059166235353 -0.023059753696741243" rpy="0 0 0"/>
     <mass value="0.9073986789846695"/>
-    <inertia ixx="0.00313" iyy="0.003181" izz="0.000211" ixy="8e-06" iyz="3.3e-05" ixz="0.000122"/>
-  </inertial>
-  <visual>
-    <origin xyz="0.11862 -0.300684 0.014775" rpy="0 0 0"/>
+    <inertia ixx="0.002786" iyy="0.003177" izz="0.00056" ixy="-2.4e-05" iyz="-1.5e-05" ixz="-0.000957"/>
+  </inertial>
+  <visual>
+    <origin xyz="0.144246 -0.197611 -0.025579" rpy="0 0 0"/>
     <geometry>
       <mesh filename="file://$(find hexapod_description)/meshes/leg_3_link_1_1.stl" scale="0.001 0.001 0.001"/>
@@ -139,5 +139,5 @@
   </visual>
   <collision>
-    <origin xyz="0.11862 -0.300684 0.014775" rpy="0 0 0"/>
+    <origin xyz="0.144246 -0.197611 -0.025579" rpy="0 0 0"/>
     <geometry>
       <mesh filename="file://$(find hexapod_description)/meshes/leg_3_link_1_1.stl" scale="0.001 0.001 0.001"/>
@@ -147,10 +147,10 @@
 <link name="leg_4_link_3_1">
   <inertial>
-    <origin xyz="0.03474109636392422 -0.003845593381223762 -0.051356732674382274" rpy="0 0 0"/>
+    <origin xyz="0.027827842510064177 0.004734636656079087 -0.05534052824142372" rpy="0 0 0"/>
     <mass value="1.0132520108724496"/>
-    <inertia ixx="0.000782" iyy="0.001231" izz="0.001141" ixy="0.000257" iyz="-0.000175" ixz="0.000456"/>
-  </inertial>
-  <visual>
-    <origin xyz="-0.178057 0.050638 -0.048896" rpy="0 0 0"/>
+    <inertia ixx="0.000814" iyy="0.001327" izz="0.001013" ixy="0.00011" iyz="-7e-05" ixz="0.000527"/>
+  </inertial>
+  <visual>
+    <origin xyz="-0.212413 0.03383 -0.035672" rpy="0 0 0"/>
     <geometry>
       <mesh filename="file://$(find hexapod_description)/meshes/leg_4_link_3_1.stl" scale="0.001 0.001 0.001"/>
@@ -159,5 +159,5 @@
   </visual>
   <collision>
-    <origin xyz="-0.178057 0.050638 -0.048896" rpy="0 0 0"/>
+    <origin xyz="-0.212413 0.03383 -0.035672" rpy="0 0 0"/>
     <geometry>
       <mesh filename="file://$(find hexapod_description)/meshes/leg_4_link_3_1.stl" scale="0.001 0.001 0.001"/>
@@ -165,12 +165,192 @@
   </collision>
 </link>
+<link name="leg_5_link_3_1">
+  <inertial>
+    <origin xyz="0.027727362528310262 0.005406300431649566 -0.05532850946625981" rpy="0 0 0"/>
+    <mass value="1.0132520108724496"/>
+    <inertia ixx="0.000808" iyy="0.001332" izz="0.001013" ixy="9.8e-05" iyz="-5.7e-05" ixz="0.000528"/>
+  </inertial>
+  <visual>
+    <origin xyz="-0.22226 -0.096026 -0.037823" rpy="0 0 0"/>
+    <geometry>
+      <mesh filename="file://$(find hexapod_description)/meshes/leg_5_link_3_1.stl" scale="0.001 0.001 0.001"/>
+    </geometry>
+    <material name="silver"/>
+  </visual>
+  <collision>
+    <origin xyz="-0.22226 -0.096026 -0.037823" rpy="0 0 0"/>
+    <geometry>
+      <mesh filename="file://$(find hexapod_description)/meshes/leg_5_link_3_1.stl" scale="0.001 0.001 0.001"/>
+    </geometry>
+  </collision>
+</link>
+<link name="leg_5_llink_2_1">
+  <inertial>
+    <origin xyz="0.03396675014480838 0.026560629165649705 0.0358235093671267" rpy="0 0 0"/>
+    <mass value="0.22866968962750417"/>
+    <inertia ixx="0.000318" iyy="0.000277" izz="0.00031" ixy="5e-06" iyz="-9e-06" ixz="-0.000127"/>
+  </inertial>
+  <visual>
+    <origin xyz="-0.291986 -0.067645 0.041757" rpy="0 0 0"/>
+    <geometry>
+      <mesh filename="file://$(find hexapod_description)/meshes/leg_5_llink_2_1.stl" scale="0.001 0.001 0.001"/>
+    </geometry>
+    <material name="silver"/>
+  </visual>
+  <collision>
+    <origin xyz="-0.291986 -0.067645 0.041757" rpy="0 0 0"/>
+    <geometry>
+      <mesh filename="file://$(find hexapod_description)/meshes/leg_5_llink_2_1.stl" scale="0.001 0.001 0.001"/>
+    </geometry>
+  </collision>
+</link>
+<link name="leg_5_link_1_1">
+  <inertial>
+    <origin xyz="0.015194262734185393 0.029558917275610747 -0.024828532452773375" rpy="0 0 0"/>
+    <mass value="0.9074869947367368"/>
+    <inertia ixx="0.002938" iyy="0.003182" izz="0.00041" ixy="1e-05" iyz="1.9e-05" ixz="0.000746"/>
+  </inertial>
+  <visual>
+    <origin xyz="-0.361611 -0.070996 -0.029944" rpy="0 0 0"/>
+    <geometry>
+      <mesh filename="file://$(find hexapod_description)/meshes/leg_5_link_1_1.stl" scale="0.001 0.001 0.001"/>
+    </geometry>
+    <material name="silver"/>
+  </visual>
+  <collision>
+    <origin xyz="-0.361611 -0.070996 -0.029944" rpy="0 0 0"/>
+    <geometry>
+      <mesh filename="file://$(find hexapod_description)/meshes/leg_5_link_1_1.stl" scale="0.001 0.001 0.001"/>
+    </geometry>
+  </collision>
+</link>
+<link name="leg_6_link_3_1">
+  <inertial>
+    <origin xyz="0.027727583128841132 0.005406596018310561 -0.055328604623189385" rpy="0 0 0"/>
+    <mass value="1.0132520108724496"/>
+    <inertia ixx="0.000808" iyy="0.001332" izz="0.001013" ixy="9.8e-05" iyz="-5.7e-05" ixz="0.000528"/>
+  </inertial>
+  <visual>
+    <origin xyz="-0.216108 -0.226108 -0.040003" rpy="0 0 0"/>
+    <geometry>
+      <mesh filename="file://$(find hexapod_description)/meshes/leg_6_link_3_1.stl" scale="0.001 0.001 0.001"/>
+    </geometry>
+    <material name="silver"/>
+  </visual>
+  <collision>
+    <origin xyz="-0.216108 -0.226108 -0.040003" rpy="0 0 0"/>
+    <geometry>
+      <mesh filename="file://$(find hexapod_description)/meshes/leg_6_link_3_1.stl" scale="0.001 0.001 0.001"/>
+    </geometry>
+  </collision>
+</link>
+<link name="leg_6_link_2_1">
+  <inertial>
+    <origin xyz="0.033966970745339664 0.02656092475231095 0.03582341421019737" rpy="0 0 0"/>
+    <mass value="0.22866968962750417"/>
+    <inertia ixx="0.000318" iyy="0.000277" izz="0.00031" ixy="5e-06" iyz="-9e-06" ixz="-0.000127"/>
+  </inertial>
+  <visual>
+    <origin xyz="-0.285834 -0.197727 0.039577" rpy="0 0 0"/>
+    <geometry>
+      <mesh filename="file://$(find hexapod_description)/meshes/leg_6_link_2_1.stl" scale="0.001 0.001 0.001"/>
+    </geometry>
+    <material name="silver"/>
+  </visual>
+  <collision>
+    <origin xyz="-0.285834 -0.197727 0.039577" rpy="0 0 0"/>
+    <geometry>
+      <mesh filename="file://$(find hexapod_description)/meshes/leg_6_link_2_1.stl" scale="0.001 0.001 0.001"/>
+    </geometry>
+  </collision>
+</link>
+<link name="leg_6_link_1_1">
+  <inertial>
+    <origin xyz="0.015193483334715818 0.029559212862271284 -0.024828627609704317" rpy="0 0 0"/>
+    <mass value="0.9074869947367368"/>
+    <inertia ixx="0.002938" iyy="0.003182" izz="0.00041" ixy="1e-05" iyz="1.9e-05" ixz="0.000746"/>
+  </inertial>
+  <visual>
+    <origin xyz="-0.35546 -0.201078 -0.032124" rpy="0 0 0"/>
+    <geometry>
+      <mesh filename="file://$(find hexapod_description)/meshes/leg_6_link_1_1.stl" scale="0.001 0.001 0.001"/>
+    </geometry>
+    <material name="silver"/>
+  </visual>
+  <collision>
+    <origin xyz="-0.35546 -0.201078 -0.032124" rpy="0 0 0"/>
+    <geometry>
+      <mesh filename="file://$(find hexapod_description)/meshes/leg_6_link_1_1.stl" scale="0.001 0.001 0.001"/>
+    </geometry>
+  </collision>
+</link>
+<link name="leg_2_link_3__1">
+  <inertial>
+    <origin xyz="-0.02799670252196973 0.004276094383967741 -0.055230856580649954" rpy="0 0 0"/>
+    <mass value="1.0126607300527286"/>
+    <inertia ixx="0.000815" iyy="0.001316" izz="0.001011" ixy="-0.000121" iyz="-8.1e-05" ixz="-0.000522"/>
+  </inertial>
+  <visual>
+    <origin xyz="0.009716 -0.099316 -0.038233" rpy="0 0 0"/>
+    <geometry>
+      <mesh filename="file://$(find hexapod_description)/meshes/leg_2_link_3__1.stl" scale="0.001 0.001 0.001"/>
+    </geometry>
+    <material name="silver"/>
+  </visual>
+  <collision>
+    <origin xyz="0.009716 -0.099316 -0.038233" rpy="0 0 0"/>
+    <geometry>
+      <mesh filename="file://$(find hexapod_description)/meshes/leg_2_link_3__1.stl" scale="0.001 0.001 0.001"/>
+    </geometry>
+  </collision>
+</link>
+<link name="leg_2_link_2_1">
+  <inertial>
+    <origin xyz="-0.03655269106835106 0.02492943001378764 0.034428145669553274" rpy="0 0 0"/>
+    <mass value="0.22871574861196214"/>
+    <inertia ixx="0.000308" iyy="0.000276" izz="0.00032" ixy="-2e-06" iyz="-3e-06" ixz="0.000128"/>
+  </inertial>
+  <visual>
+    <origin xyz="0.077653 -0.06782 0.040976" rpy="0 0 0"/>
+    <geometry>
+      <mesh filename="file://$(find hexapod_description)/meshes/leg_2_link_2_1.stl" scale="0.001 0.001 0.001"/>
+    </geometry>
+    <material name="silver"/>
+  </visual>
+  <collision>
+    <origin xyz="0.077653 -0.06782 0.040976" rpy="0 0 0"/>
+    <geometry>
+      <mesh filename="file://$(find hexapod_description)/meshes/leg_2_link_2_1.stl" scale="0.001 0.001 0.001"/>
+    </geometry>
+  </collision>
+</link>
+<link name="leg_2_link_1_1">
+  <inertial>
+    <origin xyz="-0.017401048235205913 0.028778315233383797 -0.023932405270489385" rpy="0 0 0"/>
+    <mass value="0.9073984436402253"/>
+    <inertia ixx="0.002871" iyy="0.003177" izz="0.000475" ixy="-2.3e-05" iyz="-1.6e-05" ixz="-0.000848"/>
+  </inertial>
+  <visual>
+    <origin xyz="0.150058 -0.06787 -0.027999" rpy="0 0 0"/>
+    <geometry>
+      <mesh filename="file://$(find hexapod_description)/meshes/leg_2_link_1_1.stl" scale="0.001 0.001 0.001"/>
+    </geometry>
+    <material name="silver"/>
+  </visual>
+  <collision>
+    <origin xyz="0.150058 -0.06787 -0.027999" rpy="0 0 0"/>
+    <geometry>
+      <mesh filename="file://$(find hexapod_description)/meshes/leg_2_link_1_1.stl" scale="0.001 0.001 0.001"/>
+    </geometry>
+  </collision>
+</link>
 <link name="leg_4_link_2_1">
   <inertial>
-    <origin xyz="-0.010888666203385994 0.026973289808990053 0.04744870332220183" rpy="0 0 0"/>
-    <mass value="0.2286696896275042"/>
-    <inertia ixx="0.00041" iyy="0.000283" izz="0.000211" ixy="-3e-05" iyz="-1.5e-05" ixz="7.4e-05"/>
-  </inertial>
-  <visual>
-    <origin xyz="-0.24657 0.099091 0.02152" rpy="0 0 0"/>
+    <origin xyz="0.03461242398825387 0.025734686880203556 0.03580824475570928" rpy="0 0 0"/>
+    <mass value="0.22866968962750417"/>
+    <inertia ixx="0.000318" iyy="0.000276" izz="0.00031" ixy="4e-06" iyz="-6e-06" ixz="-0.000128"/>
+  </inertial>
+  <visual>
+    <origin xyz="-0.281402 0.063887 0.043935" rpy="0 0 0"/>
     <geometry>
       <mesh filename="file://$(find hexapod_description)/meshes/leg_4_link_2_1.stl" scale="0.001 0.001 0.001"/>
@@ -179,5 +359,5 @@
   </visual>
   <collision>
-    <origin xyz="-0.24657 0.099091 0.02152" rpy="0 0 0"/>
+    <origin xyz="-0.281402 0.063887 0.043935" rpy="0 0 0"/>
     <geometry>
       <mesh filename="file://$(find hexapod_description)/meshes/leg_4_link_2_1.stl" scale="0.001 0.001 0.001"/>
@@ -187,10 +367,10 @@
 <link name="leg_4_link_1_1">
   <inertial>
-    <origin xyz="0.02172755655481845 0.024507117043729182 -0.025464522928266398" rpy="0 0 0"/>
+    <origin xyz="0.015892767008512 0.029183605213325997 -0.024836511563021524" rpy="0 0 0"/>
     <mass value="0.9074869947367368"/>
-    <inertia ixx="0.003012" iyy="0.003161" izz="0.000357" ixy="6.1e-05" iyz="-0.000166" ixz="0.000626"/>
-  </inertial>
-  <visual>
-    <origin xyz="-0.215846 0.094134 -0.073515" rpy="0 0 0"/>
+    <inertia ixx="0.002939" iyy="0.003181" izz="0.000409" ixy="1.6e-05" iyz="0.0" ixz="0.000745"/>
+  </inertial>
+  <visual>
+    <origin xyz="-0.351117 0.062215 -0.027738" rpy="0 0 0"/>
     <geometry>
       <mesh filename="file://$(find hexapod_description)/meshes/leg_4_link_1_1.stl" scale="0.001 0.001 0.001"/>
@@ -199,5 +379,5 @@
   </visual>
   <collision>
-    <origin xyz="-0.215846 0.094134 -0.073515" rpy="0 0 0"/>
+    <origin xyz="-0.351117 0.062215 -0.027738" rpy="0 0 0"/>
     <geometry>
       <mesh filename="file://$(find hexapod_description)/meshes/leg_4_link_1_1.stl" scale="0.001 0.001 0.001"/>
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
Commit message: made hexapod.xacro independed of ign_ros2_control and changed femur and tibia

File: hexapod_control/ros2_control/ros2_control.xacro (robot description, xacro)
@@ -1,4 +1,5 @@
 <?xml version="1.0" ?>
 <robot name="hexapod" xmlns:xacro="http://www.ros.org/wiki/xacro">
+<xacro:include filename="$(find hexapod_description)/urdf/hexapod.xacro" />
 <!--Ros2 control-->
 <ros2_control name="hexapod" type="system">

File: hexapod_description/urdf/hexapod.xacro (robot description, xacro)
@@ -4,5 +4,4 @@
 <xacro:include filename="$(find hexapod_description)/urdf/hexapod.trans" />
 <xacro:include filename="$(find hexapod_description)/urdf/hexapod.gazebo" />
-<xacro:include filename="$(find hexapod_control)/ros2_control/ros2_control.xacro" />
 <link name="base_link">
   <inertial>
@@ -393,5 +392,5 @@
   <dynamics damping="10" friction="0.1"/>
 </joint>
-<joint name="Leg_1_tibia" type="revolute">
+<joint name="Leg_1_femur" type="revolute">
   <origin xyz="-0.067837 -0.031701 -0.079213" rpy="0 0 0"/>
   <parent link="leg_1_link_2_1"/>
@@ -401,5 +400,5 @@
   <dynamics damping="10" friction="0.1"/>
 </joint>
-<joint name="Leg_1_femur" type="revolute">
+<joint name="Leg_1_tibia" type="revolute">
   <origin xyz="-0.072686 -0.00016 0.068679" rpy="0 0 0"/>
   <parent link="leg_1_link_3_1"/>
@@ -417,5 +416,5 @@
   <dynamics damping="10" friction="0.1"/>
 </joint>
-<joint name="Leg_3_tibia" type="revolute">
+<joint name="Leg_3_femur" type="revolute">
   <origin xyz="-0.067878 -0.031617 -0.079212" rpy="0 0 0"/>
   <parent link="leg_3_link_3_1"/>
@@ -425,5 +424,5 @@
   <dynamics damping="10" friction="0.1"/>
 </joint>
-<joint name="Leg_3_femur" type="revolute">
+<joint name="Leg_3_tibia" type="revolute">
   <origin xyz="-0.076498 5.6e-05 0.064406" rpy="0 0 0"/>
   <parent link="leg_3_link_2_1"/>
@@ -449,5 +448,5 @@
   <dynamics damping="10" friction="0.1"/>
 </joint>
-<joint name="Leg_5_tibia" type="revolute">
+<joint name="Leg_5_femur" type="revolute">
   <origin xyz="0.069726 -0.028381 -0.07958" rpy="0 0 0"/>
   <parent link="leg_5_link_3_1"/>
@@ -457,5 +456,5 @@
   <dynamics damping="10" friction="0.1"/>
 </joint>
-<joint name="Leg_5_femur" type="revolute">
+<joint name="Leg_5_tibia" type="revolute">
   <origin xyz="0.069625 0.003351 0.071701" rpy="0 0 0"/>
   <parent link="leg_5_llink_2_1"/>
@@ -473,5 +472,5 @@
   <dynamics damping="10" friction="0.1"/>
 </joint>
-<joint name="Leg_6_tibia" type="revolute">
+<joint name="Leg_6_femur" type="revolute">
   <origin xyz="0.069726 -0.028381 -0.07958" rpy="0 0 0"/>
   <parent link="leg_6_link_3_1"/>
@@ -481,5 +480,5 @@
   <dynamics damping="10" friction="0.1"/>
 </joint>
-<joint name="Leg_6_femur" type="revolute">
+<joint name="Leg_6_tibia" type="revolute">
   <origin xyz="0.069626 0.003351 0.071701" rpy="0 0 0"/>
   <parent link="leg_6_link_2_1"/>
@@ -497,5 +496,5 @@
   <dynamics damping="10" friction="0.1"/>
 </joint>
-<joint name="Leg_2_tibia" type="revolute">
+<joint name="Leg_2_femur" type="revolute">
   <origin xyz="-0.067937 -0.031496 -0.079209" rpy="0 0 0"/>
   <parent link="leg_2_link_3__1"/>
@@ -505,5 +504,5 @@
   <dynamics damping="10" friction="0.1"/>
 </joint>
-<joint name="Leg_2_femur" type="revolute">
+<joint name="Leg_2_tibia" type="revolute">
   <origin xyz="-0.072405 5e-05 0.068975" rpy="0 0 0"/>
   <parent link="leg_2_link_2_1"/>
@@ -513,5 +512,5 @@
   <dynamics damping="10" friction="0.1"/>
 </joint>
-<joint name="Leg_4_tibia" type="revolute">
+<joint name="Leg_4_femur" type="revolute">
   <origin xyz="0.068989 -0.030057 -0.079607" rpy="0 0 0"/>
   <parent link="leg_4_link_3_1"/>
@@ -521,5 +520,5 @@
   <dynamics damping="10" friction="0.1"/>
 </joint>
-<joint name="Leg_4_femur" type="revolute">
+<joint name="Leg_4_tibia" type="revolute">
   <origin xyz="0.069715 0.001672 0.071673" rpy="0 0 0"/>
   <parent link="leg_4_link_2_1"/>
