Commit message: fixed small errors

File: hexapod_control/ros2_control/ros2_control.xacro (robot description, xacro)
@@ -1,5 +1,4 @@
 <?xml version="1.0" ?>
 <robot name="hexapod" xmlns:xacro="http://www.ros.org/wiki/xacro">
-<xacro:include filename="$(find hexapod_description)/urdf/hexapod.xacro" />
 <!--Ros2 control-->
 <ros2_control name="hexapod" type="system">

File: hexapod_description/urdf/hexapod.xacro (robot description, xacro)
@@ -4,4 +4,5 @@
 <xacro:include filename="$(find hexapod_description)/urdf/hexapod.trans" />
 <xacro:include filename="$(find hexapod_description)/urdf/hexapod.gazebo" />
+<xacro:include filename="$(find hexapod_control)/ros2_control/ros2_control.xacro" />
 <link name="base_link">
   <inertial>
@@ -35,5 +36,5 @@
       <mesh filename="file://$(find hexapod_description)/meshes/leg_1_link_2_1.stl" scale="0.001 0.001 0.001"/>
     </geometry>
-    <material name="silver"/>
+    <material name="gold"/>
   </visual>
   <collision>
@@ -95,5 +96,5 @@
       <mesh filename="file://$(find hexapod_description)/meshes/leg_3_link_3_1.stl" scale="0.001 0.001 0.001"/>
     </geometry>
-    <material name="silver"/>
+    <material name="gold"/>
   </visual>
   <collision>
@@ -155,5 +156,5 @@
       <mesh filename="file://$(find hexapod_description)/meshes/leg_4_link_3_1.stl" scale="0.001 0.001 0.001"/>
     </geometry>
-    <material name="silver"/>
+    <material name="gold"/>
   </visual>
   <collision>
@@ -175,5 +176,5 @@
       <mesh filename="file://$(find hexapod_description)/meshes/leg_5_link_3_1.stl" scale="0.001 0.001 0.001"/>
     </geometry>
-    <material name="silver"/>
+    <material name="gold"/>
   </visual>
   <collision>
@@ -235,5 +236,5 @@
       <mesh filename="file://$(find hexapod_description)/meshes/leg_6_link_3_1.stl" scale="0.001 0.001 0.001"/>
     </geometry>
-    <material name="silver"/>
+    <material name="gold"/>
   </visual>
   <collision>
@@ -295,5 +296,5 @@
       <mesh filename="file://$(find hexapod_description)/meshes/leg_2_link_3__1.stl" scale="0.001 0.001 0.001"/>
     </geometry>
-    <material name="silver"/>
+    <material name="gold"/>
   </visual>
   <collision>

File: hexapod_description/urdf/materials.xacro (robot description, xacro)
@@ -2,5 +2,8 @@
 <robot name="hexapod" xmlns:xacro="http://www.ros.org/wiki/xacro" >
 <material name="silver">
-  <color rgba="1.000 0.500 0.700 1.000"/>
+  <color rgba="0.100 0.100 0.100 1.000"/>
+</material>
+<material name="gold">
+  <color rgba="0.90 0.90 0.00 1.000"/>
 </material>
 </robot>

Commit message: Changed urdf and implemented speed control

File: hexapod_control/ros2_control/ros2_control.xacro (robot description, xacro)
@@ -6,243 +6,243 @@
     <plugin>ign_ros2_control/IgnitionSystem</plugin>
   </hardware>
-  <joint name="Leg_1_coxa">
-    <command_interface name="position">
-    <param name="min">-1.57</param>
-    <param name="max">1.57</param>
-    </command_interface>
-    <state_interface name="position">
-        <param name="initial_value">0</param>
-    </state_interface>
-    <state_interface name="velocity"/>
-    <state_interface name="effort"/>
-    <limit>
-      <velocity>100.0</velocity>
-    </limit>
-  </joint>
-  <joint name="Leg_2_coxa">
-    <command_interface name="position">
-    <param name="min">-1.57</param>
-    <param name="max">1.57</param>
-    </command_interface>
-    <state_interface name="position">
-        <param name="initial_value">0</param>
-    </state_interface>
-    <state_interface name="velocity"/>
-    <state_interface name="effort"/>
-    <limit>
-      <velocity>100.0</velocity>
-    </limit>
-  </joint>
-  <joint name="Leg_3_coxa">
-    <command_interface name="position">
-    <param name="min">-1.57</param>
-    <param name="max">1.57</param>
-    </command_interface>
-    <state_interface name="position">
-        <param name="initial_value">0</param>
-    </state_interface>
-    <state_interface name="velocity"/>
-    <state_interface name="effort"/>
-    <limit>
-      <velocity>100.0</velocity>
-    </limit>
-  </joint>
-  <joint name="Leg_1_tibia">
-    <command_interface name="position">
-    <param name="min">-1.57</param>
-    <param name="max">1.57</param>
-    </command_interface>
-    <state_interface name="position">
-        <param name="initial_value">0</param>
-    </state_interface>
-    <state_interface name="velocity"/>
-    <state_interface name="effort"/>
-    <limit>
-      <velocity>100.0</velocity>
-    </limit>
-  </joint>
-  <joint name="Leg_2_tibia">
-    <command_interface name="position">
-    <param name="min">-1.57</param>
-    <param name="max">1.57</param>
-    </command_interface>
-    <state_interface name="position">
-        <param name="initial_value">0</param>
-    </state_interface>
-    <state_interface name="velocity"/>
-    <state_interface name="effort"/>
-    <limit>
-      <velocity>100.0</velocity>
-    </limit>
-  </joint>
-  <joint name="Leg_3_tibia">
-    <command_interface name="position">
-    <param name="min">-1.57</param>
-    <param name="max">1.57</param>
-    </command_interface>
-    <state_interface name="position">
-        <param name="initial_value">0</param>
-    </state_interface>
-    <state_interface name="velocity"/>
-    <state_interface name="effort"/>
-    <limit>
-      <velocity>100.0</velocity>
-    </limit>
-  </joint>
-  <joint name="Leg_1_femur">
-    <command_interface name="position">
-    <param name="min">-1.57</param>
-    <param name="max">1.57</param>
-    </command_interface>
-    <state_interface name="position">
-        <param name="initial_value">0</param>
-    </state_interface>
-    <state_interface name="velocity"/>
-    <state_interface name="effort"/>
-    <limit>
-      <velocity>100.0</velocity>
-    </limit>
-  </joint>
-  <joint name="Leg_2_femur">
-    <command_interface name="position">
-    <param name="min">-1.57</param>
-    <param name="max">1.57</param>
-    </command_interface>
-    <state_interface name="position">
-        <param name="initial_value">0</param>
-    </state_interface>
-    <state_interface name="velocity"/>
-    <state_interface name="effort"/>
-    <limit>
-      <velocity>100.0</velocity>
-    </limit>
-  </joint>
-  <joint name="Leg_3_femur">
-    <command_interface name="position">
-    <param name="min">-1.57</param>
-    <param name="max">1.57</param>
-    </command_interface>
-    <state_interface name="position">
-        <param name="initial_value">0</param>
-    </state_interface>
-    <state_interface name="velocity"/>
-    <state_interface name="effort"/>
-    <limit>
-      <velocity>100.0</velocity>
-    </limit>
-  </joint>
-  <joint name="Leg_6_femur">
-    <command_interface name="position">
-    <param name="min">-1.57</param>
-    <param name="max">1.57</param>
-    </command_interface>
-    <state_interface name="position">
-        <param name="initial_value">0</param>
-    </state_interface>
-    <state_interface name="velocity"/>
-    <state_interface name="effort"/>
-    <limit>
-      <velocity>100.0</velocity>
-    </limit>
-  </joint>
-  <joint name="Leg_4_coxa">
-    <command_interface name="position">
-    <param name="min">-1.57</param>
-    <param name="max">1.57</param>
-    </command_interface>
-    <state_interface name="position">
-        <param name="initial_value">0</param>
-    </state_interface>
-    <state_interface name="velocity"/>
-    <state_interface name="effort"/>
-    <limit>
-      <velocity>100.0</velocity>
-    </limit>
-  </joint>
-  <joint name="Leg_5_coxa">
-    <command_interface name="position">
-    <param name="min">-1.57</param>
-    <param name="max">1.57</param>
-    </command_interface>
-    <state_interface name="position">
-        <param name="initial_value">0</param>
-    </state_interface>
-    <state_interface name="velocity"/>
-    <state_interface name="effort"/>
-    <limit>
-      <velocity>100.0</velocity>
-    </limit>
-  </joint>
-  <joint name="Leg_6_coxa">
-    <command_interface name="position">
-    <param name="min">-1.57</param>
-    <param name="max">1.57</param>
-    </command_interface>
-    <state_interface name="position">
-        <param name="initial_value">0</param>
-    </state_interface>
-    <state_interface name="velocity"/>
-    <state_interface name="effort"/>
-    <limit>
-      <velocity>100.0</velocity>
-    </limit>
-  </joint>
-  <joint name="Leg_4_tibia">
-    <command_interface name="position">
-    <param name="min">-1.57</param>
-    <param name="max">1.57</param>
-    </command_interface>
-    <state_interface name="position">
-        <param name="initial_value">0</param>
-    </state_interface>
-    <state_interface name="velocity"/>
-    <state_interface name="effort"/>
-    <limit>
-      <velocity>100.0</velocity>
-    </limit>
-  </joint>
-  <joint name="Leg_5_tibia">
-    <command_interface name="position">
-    <param name="min">-1.57</param>
-    <param name="max">1.57</param>
-    </command_interface>
-    <state_interface name="position">
-        <param name="initial_value">0</param>
-    </state_interface>
-    <state_interface name="velocity"/>
-    <state_interface name="effort"/>
-    <limit>
-      <velocity>100.0</velocity>
-    </limit>
-  </joint>
-  <joint name="Leg_6_tibia">
-    <command_interface name="position">
-    <param name="min">-1.57</param>
-    <param name="max">1.57</param>
-    </command_interface>
-    <state_interface name="position">
-        <param name="initial_value">0</param>
-    </state_interface>
-    <state_interface name="velocity"/>
-    <state_interface name="effort"/>
-    <limit>
-      <velocity>100.0</velocity>
-    </limit>
-  </joint>
-  <joint name="Leg_4_femur">
-    <command_interface name="position">
-    <param name="min">-1.57</param>
-    <param name="max">1.57</param>
-    </command_interface>
-    <state_interface name="position">
-        <param name="initial_value">0</param>
-    </state_interface>
-    <state_interface name="velocity"/>
-    <state_interface name="effort"/>
-    <limit>
-      <velocity>100.0</velocity>
-    </limit>
-  </joint>
-  <joint name="Leg_5_femur">
+  <joint name="leg_1_coxa_joint">
+    <command_interface name="position">
+    <param name="min">-1.57</param>
+    <param name="max">1.57</param>
+    </command_interface>
+    <state_interface name="position">
+        <param name="initial_value">0</param>
+    </state_interface>
+    <state_interface name="velocity"/>
+    <state_interface name="effort"/>
+    <limit>
+      <velocity>100.0</velocity>
+    </limit>
+  </joint>
+  <joint name="leg_2_coxa_joint">
+    <command_interface name="position">
+    <param name="min">-1.57</param>
+    <param name="max">1.57</param>
+    </command_interface>
+    <state_interface name="position">
+        <param name="initial_value">0</param>
+    </state_interface>
+    <state_interface name="velocity"/>
+    <state_interface name="effort"/>
+    <limit>
+      <velocity>100.0</velocity>
+    </limit>
+  </joint>
+  <joint name="leg_3_coxa_joint">
+    <command_interface name="position">
+    <param name="min">-1.57</param>
+    <param name="max">1.57</param>
+    </command_interface>
+    <state_interface name="position">
+        <param name="initial_value">0</param>
+    </state_interface>
+    <state_interface name="velocity"/>
+    <state_interface name="effort"/>
+    <limit>
+      <velocity>100.0</velocity>
+    </limit>
+  </joint>
+  <joint name="leg_1_tibia_joint">
+    <command_interface name="position">
+    <param name="min">-1.57</param>
+    <param name="max">1.57</param>
+    </command_interface>
+    <state_interface name="position">
+        <param name="initial_value">0</param>
+    </state_interface>
+    <state_interface name="velocity"/>
+    <state_interface name="effort"/>
+    <limit>
+      <velocity>100.0</velocity>
+    </limit>
+  </joint>
+  <joint name="leg_2_tibia_joint">
+    <command_interface name="position">
+    <param name="min">-1.57</param>
+    <param name="max">1.57</param>
+    </command_interface>
+    <state_interface name="position">
+        <param name="initial_value">0</param>
+    </state_interface>
+    <state_interface name="velocity"/>
+    <state_interface name="effort"/>
+    <limit>
+      <velocity>100.0</velocity>
+    </limit>
+  </joint>
+  <joint name="leg_3_tibia_joint">
+    <command_interface name="position">
+    <param name="min">-1.57</param>
+    <param name="max">1.57</param>
+    </command_interface>
+    <state_interface name="position">
+        <param name="initial_value">0</param>
+    </state_interface>
+    <state_interface name="velocity"/>
+    <state_interface name="effort"/>
+    <limit>
+      <velocity>100.0</velocity>
+    </limit>
+  </joint>
+  <joint name="leg_1_femur_joint">
+    <command_interface name="position">
+    <param name="min">-1.57</param>
+    <param name="max">1.57</param>
+    </command_interface>
+    <state_interface name="position">
+        <param name="initial_value">0</param>
+    </state_interface>
+    <state_interface name="velocity"/>
+    <state_interface name="effort"/>
+    <limit>
+      <velocity>100.0</velocity>
+    </limit>
+  </joint>
+  <joint name="leg_2_femur_joint">
+    <command_interface name="position">
+    <param name="min">-1.57</param>
+    <param name="max">1.57</param>
+    </command_interface>
+    <state_interface name="position">
+        <param name="initial_value">0</param>
+    </state_interface>
+    <state_interface name="velocity"/>
+    <state_interface name="effort"/>
+    <limit>
+      <velocity>100.0</velocity>
+    </limit>
+  </joint>
+  <joint name="leg_3_femur_joint">
+    <command_interface name="position">
+    <param name="min">-1.57</param>
+    <param name="max">1.57</param>
+    </command_interface>
+    <state_interface name="position">
+        <param name="initial_value">0</param>
+    </state_interface>
+    <state_interface name="velocity"/>
+    <state_interface name="effort"/>
+    <limit>
+      <velocity>100.0</velocity>
+    </limit>
+  </joint>
+  <joint name="leg_6_femur_joint">
+    <command_interface name="position">
+    <param name="min">-1.57</param>
+    <param name="max">1.57</param>
+    </command_interface>
+    <state_interface name="position">
+        <param name="initial_value">0</param>
+    </state_interface>
+    <state_interface name="velocity"/>
+    <state_interface name="effort"/>
+    <limit>
+      <velocity>100.0</velocity>
+    </limit>
+  </joint>
+  <joint name="leg_4_coxa_joint">
+    <command_interface name="position">
+    <param name="min">-1.57</param>
+    <param name="max">1.57</param>
+    </command_interface>
+    <state_interface name="position">
+        <param name="initial_value">0</param>
+    </state_interface>
+    <state_interface name="velocity"/>
+    <state_interface name="effort"/>
+    <limit>
+      <velocity>100.0</velocity>
+    </limit>
+  </joint>
+  <joint name="leg_5_coxa_joint">
+    <command_interface name="position">
+    <param name="min">-1.57</param>
+    <param name="max">1.57</param>
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