Commit message: Changed urdf and implemented speed control

File: hexapod_description/urdf/hexapod.xacro (robot description, xacro)
@@ -25,5 +25,5 @@
   </collision>
 </link>
-<link name="leg_1_link_2_1">
+<link name="leg_1_coxa_1">
   <inertial>
     <origin xyz="-0.02800590467788834 0.004191461427254562 -0.05523214859518318" rpy="0 0 0"/>
@@ -34,25 +34,25 @@
     <origin xyz="0.003565 0.030766 -0.036053" rpy="0 0 0"/>
     <geometry>
-      <mesh filename="file://$(find hexapod_description)/meshes/leg_1_link_2_1.stl" scale="0.001 0.001 0.001"/>
-    </geometry>
-    <material name="gold"/>
+      <mesh filename="file://$(find hexapod_description)/meshes/leg_1_coxa_1.stl" scale="0.001 0.001 0.001"/>
+    </geometry>
+    <material name="silver"/>
   </visual>
   <collision>
     <origin xyz="0.003565 0.030766 -0.036053" rpy="0 0 0"/>
     <geometry>
-      <mesh filename="file://$(find hexapod_description)/meshes/leg_1_link_2_1.stl" scale="0.001 0.001 0.001"/>
-    </geometry>
-  </collision>
-</link>
-<link name="leg_1_link_3_1">
-  <inertial>
-    <origin xyz="-0.036766491881322055 0.024823115706118865 0.034277514263341684" rpy="0 0 0"/>
+      <mesh filename="file://$(find hexapod_description)/meshes/leg_1_coxa_1.stl" scale="0.001 0.001 0.001"/>
+    </geometry>
+  </collision>
+</link>
+<link name="leg_1_femur_1">
+  <inertial>
+    <origin xyz="-0.03522346741409946 0.024775287767070026 0.03589434090766965" rpy="0 0 0"/>
     <mass value="0.22871600239093776"/>
-    <inertia ixx="0.000307" iyy="0.000276" izz="0.000321" ixy="-2e-06" iyz="-2e-06" ixz="0.000128"/>
+    <inertia ixx="0.000319" iyy="0.000276" izz="0.00031" ixy="-2e-06" iyz="-2e-06" ixz="0.000128"/>
   </inertial>
   <visual>
     <origin xyz="0.071402 0.062467 0.04316" rpy="0 0 0"/>
     <geometry>
-      <mesh filename="file://$(find hexapod_description)/meshes/leg_1_link_3_1.stl" scale="0.001 0.001 0.001"/>
+      <mesh filename="file://$(find hexapod_description)/meshes/leg_1_femur_1.stl" scale="0.001 0.001 0.001"/>
     </geometry>
     <material name="silver"/>
@@ -61,29 +61,29 @@
     <origin xyz="0.071402 0.062467 0.04316" rpy="0 0 0"/>
     <geometry>
-      <mesh filename="file://$(find hexapod_description)/meshes/leg_1_link_3_1.stl" scale="0.001 0.001 0.001"/>
-    </geometry>
-  </collision>
-</link>
-<link name="leg_1_link_1_1">
-  <inertial>
-    <origin xyz="-0.01779410893760297 0.028725816249512953 -0.02370507712814386" rpy="0 0 0"/>
+      <mesh filename="file://$(find hexapod_description)/meshes/leg_1_femur_1.stl" scale="0.001 0.001 0.001"/>
+    </geometry>
+  </collision>
+</link>
+<link name="leg_1_tibia_1">
+  <inertial>
+    <origin xyz="-0.016678656476565135 0.028724980437268344 -0.024504789085526477" rpy="0 0 0"/>
     <mass value="0.907399585528797"/>
-    <inertia ixx="0.002849" iyy="0.003176" izz="0.000497" ixy="-2.4e-05" iyz="-1.8e-05" ixz="-0.000878"/>
-  </inertial>
-  <visual>
-    <origin xyz="0.144088 0.062627 -0.025519" rpy="0 0 0"/>
-    <geometry>
-      <mesh filename="file://$(find hexapod_description)/meshes/leg_1_link_1_1.stl" scale="0.001 0.001 0.001"/>
-    </geometry>
-    <material name="silver"/>
-  </visual>
-  <collision>
-    <origin xyz="0.144088 0.062627 -0.025519" rpy="0 0 0"/>
-    <geometry>
-      <mesh filename="file://$(find hexapod_description)/meshes/leg_1_link_1_1.stl" scale="0.001 0.001 0.001"/>
-    </geometry>
-  </collision>
-</link>
-<link name="leg_3_link_3_1">
+    <inertia ixx="0.002924" iyy="0.003176" izz="0.000422" ixy="-2.3e-05" iyz="-2e-05" ixz="-0.000767"/>
+  </inertial>
+  <visual>
+    <origin xyz="0.140961 0.062723 -0.028684" rpy="0 0 0"/>
+    <geometry>
+      <mesh filename="file://$(find hexapod_description)/meshes/leg_1_tibia_1.stl" scale="0.001 0.001 0.001"/>
+    </geometry>
+    <material name="silver"/>
+  </visual>
+  <collision>
+    <origin xyz="0.140961 0.062723 -0.028684" rpy="0 0 0"/>
+    <geometry>
+      <mesh filename="file://$(find hexapod_description)/meshes/leg_1_tibia_1.stl" scale="0.001 0.001 0.001"/>
+    </geometry>
+  </collision>
+</link>
+<link name="leg_3_coxa_1">
   <inertial>
     <origin xyz="-0.02800203130695705 0.004225621248029748 -0.05523202595087612" rpy="0 0 0"/>
@@ -94,25 +94,25 @@
     <origin xyz="-0.00013 -0.229172 -0.040385" rpy="0 0 0"/>
     <geometry>
-      <mesh filename="file://$(find hexapod_description)/meshes/leg_3_link_3_1.stl" scale="0.001 0.001 0.001"/>
-    </geometry>
-    <material name="gold"/>
+      <mesh filename="file://$(find hexapod_description)/meshes/leg_3_coxa_1.stl" scale="0.001 0.001 0.001"/>
+    </geometry>
+    <material name="silver"/>
   </visual>
   <collision>
     <origin xyz="-0.00013 -0.229172 -0.040385" rpy="0 0 0"/>
     <geometry>
-      <mesh filename="file://$(find hexapod_description)/meshes/leg_3_link_3_1.stl" scale="0.001 0.001 0.001"/>
-    </geometry>
-  </collision>
-</link>
-<link name="leg_3_link_2_1">
-  <inertial>
-    <origin xyz="-0.038612908125580755 0.024931950622849613 0.03209860064693253" rpy="0 0 0"/>
+      <mesh filename="file://$(find hexapod_description)/meshes/leg_3_coxa_1.stl" scale="0.001 0.001 0.001"/>
+    </geometry>
+  </collision>
+</link>
+<link name="leg_3_femur_1">
+  <inertial>
+    <origin xyz="-0.03518763654515632 0.024818021713592847 0.035899561715590445" rpy="0 0 0"/>
     <mass value="0.2287158182027981"/>
-    <inertia ixx="0.000293" iyy="0.000276" izz="0.000335" ixy="-2e-06" iyz="-3e-06" ixz="0.000126"/>
+    <inertia ixx="0.000319" iyy="0.000276" izz="0.00031" ixy="-2e-06" iyz="-2e-06" ixz="0.000128"/>
   </inertial>
   <visual>
     <origin xyz="0.067748 -0.197555 0.038827" rpy="0 0 0"/>
     <geometry>
-      <mesh filename="file://$(find hexapod_description)/meshes/leg_3_link_2_1.stl" scale="0.001 0.001 0.001"/>
+      <mesh filename="file://$(find hexapod_description)/meshes/leg_3_femur_1.stl" scale="0.001 0.001 0.001"/>
     </geometry>
     <material name="silver"/>
@@ -121,409 +121,409 @@
     <origin xyz="0.067748 -0.197555 0.038827" rpy="0 0 0"/>
     <geometry>
-      <mesh filename="file://$(find hexapod_description)/meshes/leg_3_link_2_1.stl" scale="0.001 0.001 0.001"/>
-    </geometry>
-  </collision>
-</link>
-<link name="leg_3_link_1_1">
-  <inertial>
-    <origin xyz="-0.018585545303067386 0.028750059166235353 -0.023059753696741243" rpy="0 0 0"/>
+      <mesh filename="file://$(find hexapod_description)/meshes/leg_3_femur_1.stl" scale="0.001 0.001 0.001"/>
+    </geometry>
+  </collision>
+</link>
+<link name="leg_3_tibia_1">
+  <inertial>
+    <origin xyz="-0.016646092528238454 0.028744708254966528 -0.02450268109763687" rpy="0 0 0"/>
     <mass value="0.9073986789846695"/>
-    <inertia ixx="0.002786" iyy="0.003177" izz="0.00056" ixy="-2.4e-05" iyz="-1.5e-05" ixz="-0.000957"/>
-  </inertial>
-  <visual>
-    <origin xyz="0.144246 -0.197611 -0.025579" rpy="0 0 0"/>
-    <geometry>
-      <mesh filename="file://$(find hexapod_description)/meshes/leg_3_link_1_1.stl" scale="0.001 0.001 0.001"/>
-    </geometry>
-    <material name="silver"/>
-  </visual>
-  <collision>
-    <origin xyz="0.144246 -0.197611 -0.025579" rpy="0 0 0"/>
-    <geometry>
-      <mesh filename="file://$(find hexapod_description)/meshes/leg_3_link_1_1.stl" scale="0.001 0.001 0.001"/>
-    </geometry>
-  </collision>
-</link>
-<link name="leg_4_link_3_1">
-  <inertial>
-    <origin xyz="0.027827842510064177 0.004734636656079087 -0.05534052824142372" rpy="0 0 0"/>
+    <inertia ixx="0.002924" iyy="0.003177" izz="0.000422" ixy="-2.3e-05" iyz="-1.9e-05" ixz="-0.000768"/>
+  </inertial>
+  <visual>
+    <origin xyz="0.137297 -0.197385 -0.033027" rpy="0 0 0"/>
+    <geometry>
+      <mesh filename="file://$(find hexapod_description)/meshes/leg_3_tibia_1.stl" scale="0.001 0.001 0.001"/>
+    </geometry>
+    <material name="silver"/>
+  </visual>
+  <collision>
+    <origin xyz="0.137297 -0.197385 -0.033027" rpy="0 0 0"/>
+    <geometry>
+      <mesh filename="file://$(find hexapod_description)/meshes/leg_3_tibia_1.stl" scale="0.001 0.001 0.001"/>
+    </geometry>
+  </collision>
+</link>
+<link name="leg_4_coxa_1">
+  <inertial>
+    <origin xyz="0.027993744733458475 0.0032113221383066846 -0.055366199346642296" rpy="0 0 0"/>
     <mass value="1.0132520108724496"/>
-    <inertia ixx="0.000814" iyy="0.001327" izz="0.001013" ixy="0.00011" iyz="-7e-05" ixz="0.000527"/>
+    <inertia ixx="0.000828" iyy="0.001314" izz="0.001012" ixy="0.000137" iyz="-9.9e-05" ixz="0.000522"/>
   </inertial>
   <visual>
     <origin xyz="-0.212413 0.03383 -0.035672" rpy="0 0 0"/>
     <geometry>
-      <mesh filename="file://$(find hexapod_description)/meshes/leg_4_link_3_1.stl" scale="0.001 0.001 0.001"/>
-    </geometry>
-    <material name="gold"/>
+      <mesh filename="file://$(find hexapod_description)/meshes/leg_4_coxa_1.stl" scale="0.001 0.001 0.001"/>
+    </geometry>
+    <material name="silver"/>
   </visual>
   <collision>
     <origin xyz="-0.212413 0.03383 -0.035672" rpy="0 0 0"/>
     <geometry>
-      <mesh filename="file://$(find hexapod_description)/meshes/leg_4_link_3_1.stl" scale="0.001 0.001 0.001"/>
-    </geometry>
-  </collision>
-</link>
-<link name="leg_5_link_3_1">
-  <inertial>
-    <origin xyz="0.027727362528310262 0.005406300431649566 -0.05532850946625981" rpy="0 0 0"/>
+      <mesh filename="file://$(find hexapod_description)/meshes/leg_4_coxa_1.stl" scale="0.001 0.001 0.001"/>
+    </geometry>
+  </collision>
+</link>
+<link name="leg_5_coxa_1">
+  <inertial>
+    <origin xyz="0.027997279263115404 0.00316168260604871 -0.05536637501356985" rpy="0 0 0"/>
     <mass value="1.0132520108724496"/>
-    <inertia ixx="0.000808" iyy="0.001332" izz="0.001013" ixy="9.8e-05" iyz="-5.7e-05" ixz="0.000528"/>
+    <inertia ixx="0.000828" iyy="0.001313" izz="0.001012" ixy="0.000138" iyz="-9.9e-05" ixz="0.000522"/>
   </inertial>
   <visual>
     <origin xyz="-0.22226 -0.096026 -0.037823" rpy="0 0 0"/>
     <geometry>
-      <mesh filename="file://$(find hexapod_description)/meshes/leg_5_link_3_1.stl" scale="0.001 0.001 0.001"/>
-    </geometry>
-    <material name="gold"/>
+      <mesh filename="file://$(find hexapod_description)/meshes/leg_5_coxa_1.stl" scale="0.001 0.001 0.001"/>
+    </geometry>
+    <material name="silver"/>
   </visual>
   <collision>
     <origin xyz="-0.22226 -0.096026 -0.037823" rpy="0 0 0"/>
     <geometry>
-      <mesh filename="file://$(find hexapod_description)/meshes/leg_5_link_3_1.stl" scale="0.001 0.001 0.001"/>
-    </geometry>
-  </collision>
-</link>
-<link name="leg_5_llink_2_1">
-  <inertial>
-    <origin xyz="0.03396675014480838 0.026560629165649705 0.0358235093671267" rpy="0 0 0"/>
+      <mesh filename="file://$(find hexapod_description)/meshes/leg_5_coxa_1.stl" scale="0.001 0.001 0.001"/>
+    </geometry>
+  </collision>
+</link>
+<link name="leg_5_femur_1">
+  <inertial>
+    <origin xyz="0.03603602445571802 0.02375358680070326 0.035773642331451645" rpy="0 0 0"/>
     <mass value="0.22866968962750417"/>
-    <inertia ixx="0.000318" iyy="0.000277" izz="0.00031" ixy="5e-06" iyz="-9e-06" ixz="-0.000127"/>
-  </inertial>
-  <visual>
-    <origin xyz="-0.291986 -0.067645 0.041757" rpy="0 0 0"/>
-    <geometry>
-      <mesh filename="file://$(find hexapod_description)/meshes/leg_5_llink_2_1.stl" scale="0.001 0.001 0.001"/>
-    </geometry>
-    <material name="silver"/>
-  </visual>
-  <collision>
-    <origin xyz="-0.291986 -0.067645 0.041757" rpy="0 0 0"/>
-    <geometry>
-      <mesh filename="file://$(find hexapod_description)/meshes/leg_5_llink_2_1.stl" scale="0.001 0.001 0.001"/>
-    </geometry>
-  </collision>
-</link>
-<link name="leg_5_link_1_1">
-  <inertial>
-    <origin xyz="0.015194262734185393 0.029558917275610747 -0.024828532452773375" rpy="0 0 0"/>
+    <inertia ixx="0.000318" iyy="0.000276" izz="0.00031" ixy="1e-06" iyz="1e-06" ixz="-0.000128"/>
+  </inertial>
+  <visual>
+    <origin xyz="-0.289378 -0.06214 0.041845" rpy="0 0 0"/>
+    <geometry>
+      <mesh filename="file://$(find hexapod_description)/meshes/leg_5_femur_1.stl" scale="0.001 0.001 0.001"/>
+    </geometry>
+    <material name="silver"/>
+  </visual>
+  <collision>
+    <origin xyz="-0.289378 -0.06214 0.041845" rpy="0 0 0"/>
+    <geometry>
+      <mesh filename="file://$(find hexapod_description)/meshes/leg_5_femur_1.stl" scale="0.001 0.001 0.001"/>
+    </geometry>
+  </collision>
+</link>
+<link name="leg_5_tibia_1">
+  <inertial>
+    <origin xyz="0.0174817070554254 0.02824344164925982 -0.02485431833782275" rpy="0 0 0"/>
     <mass value="0.9074869947367368"/>
-    <inertia ixx="0.002938" iyy="0.003182" izz="0.00041" ixy="1e-05" iyz="1.9e-05" ixz="0.000746"/>
-  </inertial>
-  <visual>
-    <origin xyz="-0.361611 -0.070996 -0.029944" rpy="0 0 0"/>
-    <geometry>
-      <mesh filename="file://$(find hexapod_description)/meshes/leg_5_link_1_1.stl" scale="0.001 0.001 0.001"/>
-    </geometry>
-    <material name="silver"/>
-  </visual>
-  <collision>
-    <origin xyz="-0.361611 -0.070996 -0.029944" rpy="0 0 0"/>
-    <geometry>
-      <mesh filename="file://$(find hexapod_description)/meshes/leg_5_link_1_1.stl" scale="0.001 0.001 0.001"/>
-    </geometry>
-  </collision>
-</link>
-<link name="leg_6_link_3_1">
-  <inertial>
-    <origin xyz="0.027727583128841132 0.005406596018310561 -0.055328604623189385" rpy="0 0 0"/>
+    <inertia ixx="0.002943" iyy="0.003179" izz="0.000408" ixy="3e-05" iyz="-4.2e-05" ixz="0.000741"/>
+  </inertial>
+  <visual>
+    <origin xyz="-0.359145 -0.059902 -0.029763" rpy="0 0 0"/>
+    <geometry>
+      <mesh filename="file://$(find hexapod_description)/meshes/leg_5_tibia_1.stl" scale="0.001 0.001 0.001"/>
+    </geometry>
+    <material name="silver"/>
+  </visual>
+  <collision>
+    <origin xyz="-0.359145 -0.059902 -0.029763" rpy="0 0 0"/>
+    <geometry>
+      <mesh filename="file://$(find hexapod_description)/meshes/leg_5_tibia_1.stl" scale="0.001 0.001 0.001"/>
+    </geometry>
+  </collision>
+</link>
+<link name="leg_6_coxa_1">
+  <inertial>
+    <origin xyz="0.02799749986364608 0.0031619781927097745 -0.05536647017049945" rpy="0 0 0"/>
     <mass value="1.0132520108724496"/>
-    <inertia ixx="0.000808" iyy="0.001332" izz="0.001013" ixy="9.8e-05" iyz="-5.7e-05" ixz="0.000528"/>
+    <inertia ixx="0.000828" iyy="0.001313" izz="0.001012" ixy="0.000138" iyz="-9.9e-05" ixz="0.000522"/>
   </inertial>
   <visual>
     <origin xyz="-0.216108 -0.226108 -0.040003" rpy="0 0 0"/>
     <geometry>
-      <mesh filename="file://$(find hexapod_description)/meshes/leg_6_link_3_1.stl" scale="0.001 0.001 0.001"/>
-    </geometry>
-    <material name="gold"/>
+      <mesh filename="file://$(find hexapod_description)/meshes/leg_6_coxa_1.stl" scale="0.001 0.001 0.001"/>
+    </geometry>
+    <material name="silver"/>
   </visual>
   <collision>
     <origin xyz="-0.216108 -0.226108 -0.040003" rpy="0 0 0"/>
     <geometry>
-      <mesh filename="file://$(find hexapod_description)/meshes/leg_6_link_3_1.stl" scale="0.001 0.001 0.001"/>
-    </geometry>
-  </collision>
-</link>
-<link name="leg_6_link_2_1">
-  <inertial>
-    <origin xyz="0.033966970745339664 0.02656092475231095 0.03582341421019737" rpy="0 0 0"/>
+      <mesh filename="file://$(find hexapod_description)/meshes/leg_6_coxa_1.stl" scale="0.001 0.001 0.001"/>
+    </geometry>
+  </collision>
+</link>
+<link name="leg_6_femur_1">
+  <inertial>
+    <origin xyz="0.036035245056249054 0.023753882387363978 0.035773547174522295" rpy="0 0 0"/>
     <mass value="0.22866968962750417"/>
-    <inertia ixx="0.000318" iyy="0.000277" izz="0.00031" ixy="5e-06" iyz="-9e-06" ixz="-0.000127"/>
-  </inertial>
-  <visual>
-    <origin xyz="-0.285834 -0.197727 0.039577" rpy="0 0 0"/>
-    <geometry>
-      <mesh filename="file://$(find hexapod_description)/meshes/leg_6_link_2_1.stl" scale="0.001 0.001 0.001"/>
-    </geometry>
-    <material name="silver"/>
-  </visual>
-  <collision>
-    <origin xyz="-0.285834 -0.197727 0.039577" rpy="0 0 0"/>
-    <geometry>
-      <mesh filename="file://$(find hexapod_description)/meshes/leg_6_link_2_1.stl" scale="0.001 0.001 0.001"/>
-    </geometry>
-  </collision>
-</link>
-<link name="leg_6_link_1_1">
-  <inertial>
-    <origin xyz="0.015193483334715818 0.029559212862271284 -0.024828627609704317" rpy="0 0 0"/>
+    <inertia ixx="0.000318" iyy="0.000276" izz="0.00031" ixy="1e-06" iyz="1e-06" ixz="-0.000128"/>
+  </inertial>
+  <visual>
+    <origin xyz="-0.283227 -0.192222 0.039665" rpy="0 0 0"/>
+    <geometry>
+      <mesh filename="file://$(find hexapod_description)/meshes/leg_6_femur_1.stl" scale="0.001 0.001 0.001"/>
+    </geometry>
+    <material name="silver"/>
+  </visual>
+  <collision>
+    <origin xyz="-0.283227 -0.192222 0.039665" rpy="0 0 0"/>
+    <geometry>
+      <mesh filename="file://$(find hexapod_description)/meshes/leg_6_femur_1.stl" scale="0.001 0.001 0.001"/>
+    </geometry>
+  </collision>
+</link>
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
File: hexapod_description/urdf/materials.xacro (robot description, xacro)
@@ -2,8 +2,5 @@
 <robot name="hexapod" xmlns:xacro="http://www.ros.org/wiki/xacro" >
 <material name="silver">
-  <color rgba="0.100 0.100 0.100 1.000"/>
-</material>
-<material name="gold">
-  <color rgba="0.90 0.90 0.00 1.000"/>
+  <color rgba="0.700 0.700 0.700 1.000"/>
 </material>
 </robot>
