Commit message: changed to revolute joints

File: hexapod_description/urdf/hexapod.xacro (robot description, xacro)
@@ -384,5 +384,5 @@
   </collision>
 </link>
-<joint name="Revolute 63" type="continuous">
+<joint name="Revolute 63" type="revolute">
   <origin xyz="-0.031628 -0.00646 0.021757" rpy="0 0 0"/>
   <parent link="base_link"/>
@@ -392,5 +392,5 @@
   <dynamics damping="10" friction="0.1"/>
 </joint>
-<joint name="Revolute 64" type="continuous">
+<joint name="Revolute 64" type="revolute">
   <origin xyz="-0.049275 -0.046824 -0.085212" rpy="0 0 0"/>
   <parent link="leg_1_link_2_1"/>
@@ -400,5 +400,5 @@
   <dynamics damping="10" friction="0.1"/>
 </joint>
-<joint name="Revolute 65" type="continuous">
+<joint name="Revolute 65" type="revolute">
   <origin xyz="-0.094492 -0.016959 0.027993" rpy="0 0 0"/>
   <parent link="leg_1_link_3_1"/>
@@ -408,5 +408,5 @@
   <dynamics damping="10" friction="0.1"/>
 </joint>
-<joint name="Revolute 69" type="continuous">
+<joint name="Revolute 69" type="revolute">
   <origin xyz="0.02145 0.24803 0.025922" rpy="0 0 0"/>
   <parent link="base_link"/>
@@ -416,5 +416,5 @@
   <dynamics damping="10" friction="0.1"/>
 </joint>
-<joint name="Revolute 70" type="continuous">
+<joint name="Revolute 70" type="revolute">
   <origin xyz="-0.064347 0.007284 -0.087681" rpy="0 0 0"/>
   <parent link="leg_3_link_3_1"/>
@@ -424,5 +424,5 @@
   <dynamics damping="10" friction="0.1"/>
 </joint>
-<joint name="Revolute 71" type="continuous">
+<joint name="Revolute 71" type="revolute">
   <origin xyz="-0.075723 0.04537 0.046984" rpy="0 0 0"/>
   <parent link="leg_3_link_2_1"/>
@@ -432,5 +432,5 @@
   <dynamics damping="10" friction="0.1"/>
 </joint>
-<joint name="Revolute 72" type="continuous">
+<joint name="Revolute 72" type="revolute">
   <origin xyz="0.178057 -0.050638 0.048896" rpy="0 0 0"/>
   <parent link="base_link"/>
@@ -440,5 +440,5 @@
   <dynamics damping="10" friction="0.1"/>
 </joint>
-<joint name="Revolute 73" type="continuous">
+<joint name="Revolute 73" type="revolute">
   <origin xyz="0.068513 -0.048453 -0.070416" rpy="0 0 0"/>
   <parent link="leg_4_link_3_1"/>
@@ -448,5 +448,5 @@
   <dynamics damping="10" friction="0.1"/>
 </joint>
-<joint name="Revolute 74" type="continuous">
+<joint name="Revolute 74" type="revolute">
   <origin xyz="-0.030724 0.004957 0.095035" rpy="0 0 0"/>
   <parent link="leg_4_link_2_1"/>
@@ -456,5 +456,5 @@
   <dynamics damping="10" friction="0.1"/>
 </joint>
-<joint name="Revolute 75" type="continuous">
+<joint name="Revolute 75" type="revolute">
   <origin xyz="0.212362 0.074971 0.051984" rpy="0 0 0"/>
   <parent link="base_link"/>
@@ -464,5 +464,5 @@
   <dynamics damping="10" friction="0.1"/>
 </joint>
-<joint name="Revolute 76" type="continuous">
+<joint name="Revolute 76" type="revolute">
   <origin xyz="0.063891 -0.053704 -0.070951" rpy="0 0 0"/>
   <parent link="leg_5_link_3_1"/>
@@ -472,5 +472,5 @@
   <dynamics damping="10" friction="0.1"/>
 </joint>
-<joint name="Revolute 77" type="continuous">
+<joint name="Revolute 77" type="revolute">
   <origin xyz="0.020996 -0.009438 0.097315" rpy="0 0 0"/>
   <parent link="leg_5_llink_2_1"/>
@@ -480,5 +480,5 @@
   <dynamics damping="10" friction="0.1"/>
 </joint>
-<joint name="Revolute 78" type="continuous">
+<joint name="Revolute 78" type="revolute">
   <origin xyz="0.231135 0.203852 0.053061" rpy="0 0 0"/>
   <parent link="base_link"/>
@@ -488,5 +488,5 @@
   <dynamics damping="10" friction="0.1"/>
 </joint>
-<joint name="Revolute 79" type="continuous">
+<joint name="Revolute 79" type="revolute">
   <origin xyz="0.069208 -0.047573 -0.070336" rpy="0 0 0"/>
   <parent link="leg_6_link_3_1"/>
@@ -496,5 +496,5 @@
   <dynamics damping="10" friction="0.1"/>
 </joint>
-<joint name="Revolute 80" type="continuous">
+<joint name="Revolute 80" type="revolute">
   <origin xyz="0.065727 -0.014193 0.074017" rpy="0 0 0"/>
   <parent link="leg_6_link_2_1"/>
@@ -504,5 +504,5 @@
   <dynamics damping="10" friction="0.1"/>
 </joint>
-<joint name="Revolute 81" type="continuous">
+<joint name="Revolute 81" type="revolute">
   <origin xyz="-0.012855 0.122421 0.022834" rpy="0 0 0"/>
   <parent link="base_link"/>
@@ -512,5 +512,5 @@
   <dynamics damping="10" friction="0.1"/>
 </joint>
-<joint name="Revolute 82" type="continuous">
+<joint name="Revolute 82" type="revolute">
   <origin xyz="-0.059269 -0.029299 -0.086662" rpy="0 0 0"/>
   <parent link="leg_2_link_3__1__1"/>
@@ -520,5 +520,5 @@
   <dynamics damping="10" friction="0.1"/>
 </joint>
-<joint name="Revolute 83" type="continuous">
+<joint name="Revolute 83" type="revolute">
   <origin xyz="-0.09777 0.007821 0.019488" rpy="0 0 0"/>
   <parent link="leg_2_link_2_1"/>

Commit message: ros2 control

File: hexapod_description/urdf/hexapod.xacro (robot description, xacro)
@@ -384,5 +384,5 @@
   </collision>
 </link>
-<joint name="Revolute 63" type="revolute">
+<joint name="Revolute_63" type="revolute">
   <origin xyz="-0.031628 -0.00646 0.021757" rpy="0 0 0"/>
   <parent link="base_link"/>
@@ -392,5 +392,5 @@
   <dynamics damping="10" friction="0.1"/>
 </joint>
-<joint name="Revolute 64" type="revolute">
+<joint name="Revolute_64" type="revolute">
   <origin xyz="-0.049275 -0.046824 -0.085212" rpy="0 0 0"/>
   <parent link="leg_1_link_2_1"/>
@@ -400,5 +400,5 @@
   <dynamics damping="10" friction="0.1"/>
 </joint>
-<joint name="Revolute 65" type="revolute">
+<joint name="Revolute_65" type="revolute">
   <origin xyz="-0.094492 -0.016959 0.027993" rpy="0 0 0"/>
   <parent link="leg_1_link_3_1"/>
@@ -408,5 +408,5 @@
   <dynamics damping="10" friction="0.1"/>
 </joint>
-<joint name="Revolute 69" type="revolute">
+<joint name="Revolute_69" type="revolute">
   <origin xyz="0.02145 0.24803 0.025922" rpy="0 0 0"/>
   <parent link="base_link"/>
@@ -416,5 +416,5 @@
   <dynamics damping="10" friction="0.1"/>
 </joint>
-<joint name="Revolute 70" type="revolute">
+<joint name="Revolute_70" type="revolute">
   <origin xyz="-0.064347 0.007284 -0.087681" rpy="0 0 0"/>
   <parent link="leg_3_link_3_1"/>
@@ -424,5 +424,5 @@
   <dynamics damping="10" friction="0.1"/>
 </joint>
-<joint name="Revolute 71" type="revolute">
+<joint name="Revolute_71" type="revolute">
   <origin xyz="-0.075723 0.04537 0.046984" rpy="0 0 0"/>
   <parent link="leg_3_link_2_1"/>
@@ -432,5 +432,5 @@
   <dynamics damping="10" friction="0.1"/>
 </joint>
-<joint name="Revolute 72" type="revolute">
+<joint name="Revolute_72" type="revolute">
   <origin xyz="0.178057 -0.050638 0.048896" rpy="0 0 0"/>
   <parent link="base_link"/>
@@ -440,5 +440,5 @@
   <dynamics damping="10" friction="0.1"/>
 </joint>
-<joint name="Revolute 73" type="revolute">
+<joint name="Revolute_73" type="revolute">
   <origin xyz="0.068513 -0.048453 -0.070416" rpy="0 0 0"/>
   <parent link="leg_4_link_3_1"/>
@@ -448,5 +448,5 @@
   <dynamics damping="10" friction="0.1"/>
 </joint>
-<joint name="Revolute 74" type="revolute">
+<joint name="Revolute_74" type="revolute">
   <origin xyz="-0.030724 0.004957 0.095035" rpy="0 0 0"/>
   <parent link="leg_4_link_2_1"/>
@@ -456,5 +456,5 @@
   <dynamics damping="10" friction="0.1"/>
 </joint>
-<joint name="Revolute 75" type="revolute">
+<joint name="Revolute_75" type="revolute">
   <origin xyz="0.212362 0.074971 0.051984" rpy="0 0 0"/>
   <parent link="base_link"/>
@@ -464,5 +464,5 @@
   <dynamics damping="10" friction="0.1"/>
 </joint>
-<joint name="Revolute 76" type="revolute">
+<joint name="Revolute_76" type="revolute">
   <origin xyz="0.063891 -0.053704 -0.070951" rpy="0 0 0"/>
   <parent link="leg_5_link_3_1"/>
@@ -472,5 +472,5 @@
   <dynamics damping="10" friction="0.1"/>
 </joint>
-<joint name="Revolute 77" type="revolute">
+<joint name="Revolute_77" type="revolute">
   <origin xyz="0.020996 -0.009438 0.097315" rpy="0 0 0"/>
   <parent link="leg_5_llink_2_1"/>
@@ -480,5 +480,5 @@
   <dynamics damping="10" friction="0.1"/>
 </joint>
-<joint name="Revolute 78" type="revolute">
+<joint name="Revolute_78" type="revolute">
   <origin xyz="0.231135 0.203852 0.053061" rpy="0 0 0"/>
   <parent link="base_link"/>
@@ -488,5 +488,5 @@
   <dynamics damping="10" friction="0.1"/>
 </joint>
-<joint name="Revolute 79" type="revolute">
+<joint name="Revolute_79" type="revolute">
   <origin xyz="0.069208 -0.047573 -0.070336" rpy="0 0 0"/>
   <parent link="leg_6_link_3_1"/>
@@ -496,5 +496,5 @@
   <dynamics damping="10" friction="0.1"/>
 </joint>
-<joint name="Revolute 80" type="revolute">
+<joint name="Revolute_80" type="revolute">
   <origin xyz="0.065727 -0.014193 0.074017" rpy="0 0 0"/>
   <parent link="leg_6_link_2_1"/>
@@ -504,5 +504,5 @@
   <dynamics damping="10" friction="0.1"/>
 </joint>
-<joint name="Revolute 81" type="revolute">
+<joint name="Revolute_81" type="revolute">
   <origin xyz="-0.012855 0.122421 0.022834" rpy="0 0 0"/>
   <parent link="base_link"/>
@@ -512,5 +512,5 @@
   <dynamics damping="10" friction="0.1"/>
 </joint>
-<joint name="Revolute 82" type="revolute">
+<joint name="Revolute_82" type="revolute">
   <origin xyz="-0.059269 -0.029299 -0.086662" rpy="0 0 0"/>
   <parent link="leg_2_link_3__1__1"/>
@@ -520,5 +520,5 @@
   <dynamics damping="10" friction="0.1"/>
 </joint>
-<joint name="Revolute 83" type="revolute">
+<joint name="Revolute_83" type="revolute">
   <origin xyz="-0.09777 0.007821 0.019488" rpy="0 0 0"/>
   <parent link="leg_2_link_2_1"/>
@@ -528,3 +528,176 @@
   <dynamics damping="10" friction="0.1"/>
 </joint>
+<!--Ros2 control-->
+<ros2_control name="hexapod" type="system">
+  <hardware>
+    <plugin>ign_ros2_control/IgnitionSystem</plugin>
+  </hardware>
+  <joint name="Revolute_63">
+    <command_interface name="position">
+    <param name="min">-1</param>
+    <param name="max">1</param>
+    </command_interface>
+    <state_interface name="position">
+      <param name="initial_value">0</param>
+    </state_interface>
+  </joint>
+  <joint name="Revolute_64">
+    <command_interface name="position">
+    <param name="min">-1</param>
+    <param name="max">1</param>
+    </command_interface>
+    <state_interface name="position">
+      <param name="initial_value">0</param>
+    </state_interface>
+  </joint>
+  <joint name="Revolute_65">
+    <command_interface name="position">
+    <param name="min">-1</param>
+    <param name="max">1</param>
+    </command_interface>
+    <state_interface name="position">
+      <param name="initial_value">0</param>
+    </state_interface>
+  </joint>
+  <joint name="Revolute_69">
+    <command_interface name="position">
+    <param name="min">-1</param>
+    <param name="max">1</param>
+    </command_interface>
+    <state_interface name="position">
+      <param name="initial_value">0</param>
+    </state_interface>
+  </joint>
+  <joint name="Revolute_70">
+    <command_interface name="position">
+    <param name="min">-1</param>
+    <param name="max">1</param>
+    </command_interface>
+    <state_interface name="position">
+      <param name="initial_value">0</param>
+    </state_interface>
+  </joint>
+  <joint name="Revolute_71">
+    <command_interface name="position">
+    <param name="min">-1</param>
+    <param name="max">1</param>
+    </command_interface>
+    <state_interface name="position">
+      <param name="initial_value">0</param>
+    </state_interface>
+  </joint>
+  <joint name="Revolute_72">
+    <command_interface name="position">
+    <param name="min">-1</param>
+    <param name="max">1</param>
+    </command_interface>
+    <state_interface name="position">
+      <param name="initial_value">0</param>
+    </state_interface>
+  </joint>
+  <joint name="Revolute_73">
+    <command_interface name="position">
+    <param name="min">-1</param>
+    <param name="max">1</param>
+    </command_interface>
+    <state_interface name="position">
+      <param name="initial_value">0</param>
+    </state_interface>
+  </joint>
+  <joint name="Revolute_74">
+    <command_interface name="position">
+    <param name="min">-1</param>
+    <param name="max">1</param>
+    </command_interface>
+    <state_interface name="position">
+      <param name="initial_value">0</param>
+    </state_interface>
+  </joint>
+  <joint name="Revolute_75">
+    <command_interface name="position">
+    <param name="min">-1</param>
+    <param name="max">1</param>
+    </command_interface>
+    <state_interface name="position">
+      <param name="initial_value">0</param>
+    </state_interface>
+  </joint>
+  <joint name="Revolute_76">
+    <command_interface name="position">
+    <param name="min">-1</param>
+    <param name="max">1</param>
+    </command_interface>
+    <state_interface name="position">
+      <param name="initial_value">0</param>
+    </state_interface>
+  </joint>
+  <joint name="Revolute_77">
+    <command_interface name="position">
+    <param name="min">-1</param>
+    <param name="max">1</param>
+    </command_interface>
+    <state_interface name="position">
+      <param name="initial_value">0</param>
+    </state_interface>
+  </joint>
+  <joint name="Revolute_78">
+    <command_interface name="position">
+    <param name="min">-1</param>
+    <param name="max">1</param>
+    </command_interface>
+    <state_interface name="position">
+      <param name="initial_value">0</param>
+    </state_interface>
+  </joint>
+  <joint name="Revolute_79">
+    <command_interface name="position">
+    <param name="min">-1</param>
+    <param name="max">1</param>
+    </command_interface>
+    <state_interface name="position">
+      <param name="initial_value">0</param>
+    </state_interface>
+  </joint>
+  <joint name="Revolute_80">
+    <command_interface name="position">
+    <param name="min">-1</param>
+    <param name="max">1</param>
+    </command_interface>
+    <state_interface name="position">
+      <param name="initial_value">0</param>
+    </state_interface>
+  </joint>
+  <joint name="Revolute_81">
+    <command_interface name="position">
+    <param name="min">-1</param>
+    <param name="max">1</param>
+    </command_interface>
+    <state_interface name="position">
+      <param name="initial_value">0</param>
+    </state_interface>
+  </joint>
+  <joint name="Revolute_82">
+    <command_interface name="position">
+    <param name="min">-1</param>
+    <param name="max">1</param>
+    </command_interface>
+    <state_interface name="position">
+      <param name="initial_value">0</param>
+    </state_interface>
+  </joint>
+  <joint name="Revolute_83">
+    <command_interface name="position">
+    <param name="min">-1</param>
+    <param name="max">1</param>
+    </command_interface>
+    <state_interface name="position">
+      <param name="initial_value">0</param>
+    </state_interface>
+  </joint>
+</ros2_control>
+<gazebo>
+  <plugin filename="ign_ros2_control-system" name="ign_ros2_control::IgnitionROS2ControlPlugin">
+    <parameters>$(find hexapod_description)/config/hexapod_controller.yaml</parameters>
+  </plugin>
+</gazebo>
 </robot>

Commit message: created ros_control package

File: hexapod_description/urdf/hexapod.xacro (robot description, xacro)
@@ -4,4 +4,5 @@
 <xacro:include filename="$(find hexapod_description)/urdf/hexapod.trans" />
 <xacro:include filename="$(find hexapod_description)/urdf/hexapod.gazebo" />
+<xacro:include filename="$(find hexapod_control)/ros2_control/ros2_control.xacro" />
 <link name="base_link">
   <inertial>
@@ -528,176 +529,3 @@
   <dynamics damping="10" friction="0.1"/>
 </joint>
-<!--Ros2 control-->
-<ros2_control name="hexapod" type="system">
-  <hardware>
-    <plugin>ign_ros2_control/IgnitionSystem</plugin>
-  </hardware>
-  <joint name="Revolute_63">
-    <command_interface name="position">
-    <param name="min">-1</param>
-    <param name="max">1</param>
-    </command_interface>
-    <state_interface name="position">
-      <param name="initial_value">0</param>
-    </state_interface>
-  </joint>
-  <joint name="Revolute_64">
-    <command_interface name="position">
-    <param name="min">-1</param>
-    <param name="max">1</param>
-    </command_interface>
-    <state_interface name="position">
-      <param name="initial_value">0</param>
-    </state_interface>
-  </joint>
-  <joint name="Revolute_65">
-    <command_interface name="position">
-    <param name="min">-1</param>
-    <param name="max">1</param>
-    </command_interface>
-    <state_interface name="position">
-      <param name="initial_value">0</param>
-    </state_interface>
-  </joint>
-  <joint name="Revolute_69">
-    <command_interface name="position">
-    <param name="min">-1</param>
-    <param name="max">1</param>
-    </command_interface>
-    <state_interface name="position">
-      <param name="initial_value">0</param>
-    </state_interface>
-  </joint>
-  <joint name="Revolute_70">
-    <command_interface name="position">
-    <param name="min">-1</param>
-    <param name="max">1</param>
-    </command_interface>
-    <state_interface name="position">
-      <param name="initial_value">0</param>
-    </state_interface>
-  </joint>
-  <joint name="Revolute_71">
-    <command_interface name="position">
-    <param name="min">-1</param>
-    <param name="max">1</param>
-    </command_interface>
-    <state_interface name="position">
-      <param name="initial_value">0</param>
-    </state_interface>
-  </joint>
-  <joint name="Revolute_72">
-    <command_interface name="position">
-    <param name="min">-1</param>
-    <param name="max">1</param>
-    </command_interface>
-    <state_interface name="position">
-      <param name="initial_value">0</param>
-    </state_interface>
-  </joint>
-  <joint name="Revolute_73">
-    <command_interface name="position">
-    <param name="min">-1</param>
-    <param name="max">1</param>
-    </command_interface>
-    <state_interface name="position">
-      <param name="initial_value">0</param>
-    </state_interface>
-  </joint>
-  <joint name="Revolute_74">
-    <command_interface name="position">
-    <param name="min">-1</param>
-    <param name="max">1</param>
-    </command_interface>
-    <state_interface name="position">
-      <param name="initial_value">0</param>
-    </state_interface>
-  </joint>
-  <joint name="Revolute_75">
-    <command_interface name="position">
-    <param name="min">-1</param>
-    <param name="max">1</param>
-    </command_interface>
-    <state_interface name="position">
-      <param name="initial_value">0</param>
-    </state_interface>
-  </joint>
-  <joint name="Revolute_76">
-    <command_interface name="position">
-    <param name="min">-1</param>
-    <param name="max">1</param>
-    </command_interface>
-    <state_interface name="position">
-      <param name="initial_value">0</param>
-    </state_interface>
-  </joint>
-  <joint name="Revolute_77">
-    <command_interface name="position">
-    <param name="min">-1</param>
-    <param name="max">1</param>
-    </command_interface>
-    <state_interface name="position">
-      <param name="initial_value">0</param>
-    </state_interface>
-  </joint>
-  <joint name="Revolute_78">
-    <command_interface name="position">
-    <param name="min">-1</param>
-    <param name="max">1</param>
-    </command_interface>
-    <state_interface name="position">
-      <param name="initial_value">0</param>
-    </state_interface>
-  </joint>
-  <joint name="Revolute_79">
-    <command_interface name="position">
-    <param name="min">-1</param>
-    <param name="max">1</param>
-    </command_interface>
-    <state_interface name="position">
-      <param name="initial_value">0</param>
-    </state_interface>
-  </joint>
-  <joint name="Revolute_80">
-    <command_interface name="position">
-    <param name="min">-1</param>
-    <param name="max">1</param>
-    </command_interface>
-    <state_interface name="position">
-      <param name="initial_value">0</param>
-    </state_interface>
-  </joint>
-  <joint name="Revolute_81">
-    <command_interface name="position">
-    <param name="min">-1</param>
-    <param name="max">1</param>
-    </command_interface>
-    <state_interface name="position">
-      <param name="initial_value">0</param>
-    </state_interface>
-  </joint>
-  <joint name="Revolute_82">
-    <command_interface name="position">
-    <param name="min">-1</param>
-    <param name="max">1</param>
-    </command_interface>
-    <state_interface name="position">
-      <param name="initial_value">0</param>
-    </state_interface>
-  </joint>
-  <joint name="Revolute_83">
-    <command_interface name="position">
-    <param name="min">-1</param>
-    <param name="max">1</param>
-    </command_interface>
-    <state_interface name="position">
-      <param name="initial_value">0</param>
-    </state_interface>
-  </joint>
-</ros2_control>
-<gazebo>
-  <plugin filename="ign_ros2_control-system" name="ign_ros2_control::IgnitionROS2ControlPlugin">
-    <parameters>$(find hexapod_description)/config/hexapod_controller.yaml</parameters>
-  </plugin>
-</gazebo>
 </robot>
