Commit message: changed bot controller

File: hexapod_description/urdf/hexapod.xacro (robot description, xacro)
@@ -390,5 +390,5 @@
   <child link="leg_1_link_2_1"/>
   <axis xyz="0.126261 -0.010099 -0.991946"/>
-  <limit effort="100" lower="-1.57" upper="1.57" velocity="100"/>
+  <limit effort="100" lower="-1.57" upper="1.57" velocity="1"/>
   <dynamics damping="10" friction="0.1"/>
 </joint>
@@ -398,5 +398,5 @@
   <child link="leg_1_link_3_1"/>
   <axis xyz="0.186207 -0.981932 0.033699"/>
-  <limit effort="100" lower="-1.57" upper="1.57" velocity="100"/>
+  <limit effort="100" lower="-1.57" upper="1.57" velocity="1"/>
   <dynamics damping="10" friction="0.1"/>
 </joint>
@@ -406,5 +406,5 @@
   <child link="leg_1_link_1_1"/>
   <axis xyz="0.186207 -0.981932 0.033699"/>
-  <limit effort="100" lower="-1.57" upper="1.57" velocity="100"/>
+  <limit effort="100" lower="-1.57" upper="1.57" velocity="1"/>
   <dynamics damping="10" friction="0.1"/>
 </joint>
@@ -414,5 +414,5 @@
   <child link="leg_3_link_3_1"/>
   <axis xyz="0.126261 -0.010099 -0.991946"/>
-  <limit effort="100" lower="-1.57" upper="1.57" velocity="100"/>
+  <limit effort="100" lower="-1.57" upper="1.57" velocity="1"/>
   <dynamics damping="10" friction="0.1"/>
 </joint>
@@ -422,5 +422,5 @@
   <child link="leg_3_link_2_1"/>
   <axis xyz="-0.540263 -0.839339 -0.060222"/>
-  <limit effort="100" lower="-1.57" upper="1.57" velocity="100"/>
+  <limit effort="100" lower="-1.57" upper="1.57" velocity="1"/>
   <dynamics damping="10" friction="0.1"/>
 </joint>
@@ -430,5 +430,5 @@
   <child link="leg_3_link_1_1"/>
   <axis xyz="-0.540263 -0.839339 -0.060222"/>
-  <limit effort="100" lower="-1.57" upper="1.57" velocity="100"/>
+  <limit effort="100" lower="-1.57" upper="1.57" velocity="1"/>
   <dynamics damping="10" friction="0.1"/>
 </joint>
@@ -438,5 +438,5 @@
   <child link="leg_4_link_3_1"/>
   <axis xyz="0.126261 -0.010099 -0.991946"/>
-  <limit effort="100" lower="-1.57" upper="1.57" velocity="100"/>
+  <limit effort="100" lower="-1.57" upper="1.57" velocity="1"/>
   <dynamics damping="10" friction="0.1"/>
 </joint>
@@ -446,5 +446,5 @@
   <child link="leg_4_link_2_1"/>
   <axis xyz="-0.209414 -0.977684 -0.016701"/>
-  <limit effort="100" lower="-1.57" upper="1.57" velocity="100"/>
+  <limit effort="100" lower="-1.57" upper="1.57" velocity="1"/>
   <dynamics damping="10" friction="0.1"/>
 </joint>
@@ -454,5 +454,5 @@
   <child link="leg_4_link_1_1"/>
   <axis xyz="0.209414 0.977684 0.016701"/>
-  <limit effort="100" lower="-1.57" upper="1.57" velocity="100"/>
+  <limit effort="100" lower="-1.57" upper="1.57" velocity="1"/>
   <dynamics damping="10" friction="0.1"/>
 </joint>
@@ -462,5 +462,5 @@
   <child link="leg_5_link_3_1"/>
   <axis xyz="0.126261 -0.010099 -0.991946"/>
-  <limit effort="100" lower="-1.57" upper="1.57" velocity="100"/>
+  <limit effort="100" lower="-1.57" upper="1.57" velocity="1"/>
   <dynamics damping="10" friction="0.1"/>
 </joint>
@@ -470,5 +470,5 @@
   <child link="leg_5_llink_2_1"/>
   <axis xyz="-0.298057 -0.954131 -0.028224"/>
-  <limit effort="100" lower="-1.57" upper="1.57" velocity="100"/>
+  <limit effort="100" lower="-1.57" upper="1.57" velocity="1"/>
   <dynamics damping="10" friction="0.1"/>
 </joint>
@@ -478,5 +478,5 @@
   <child link="leg_5_link_1_1"/>
   <axis xyz="0.298057 0.954131 0.028224"/>
-  <limit effort="100" lower="-1.57" upper="1.57" velocity="100"/>
+  <limit effort="100" lower="-1.57" upper="1.57" velocity="1"/>
   <dynamics damping="10" friction="0.1"/>
 </joint>
@@ -486,5 +486,5 @@
   <child link="leg_6_link_3_1"/>
   <axis xyz="0.126261 -0.010099 -0.991946"/>
-  <limit effort="100" lower="-1.57" upper="1.57" velocity="100"/>
+  <limit effort="100" lower="-1.57" upper="1.57" velocity="1"/>
   <dynamics damping="10" friction="0.1"/>
 </joint>
@@ -494,5 +494,5 @@
   <child link="leg_6_link_2_1"/>
   <axis xyz="-0.195044 -0.980682 -0.014842"/>
-  <limit effort="100" lower="-1.57" upper="1.57" velocity="100"/>
+  <limit effort="100" lower="-1.57" upper="1.57" velocity="1"/>
   <dynamics damping="10" friction="0.1"/>
 </joint>
@@ -502,5 +502,5 @@
   <child link="leg_6_link_1_1"/>
   <axis xyz="0.195044 0.980682 0.014842"/>
-  <limit effort="100" lower="-1.57" upper="1.57" velocity="100"/>
+  <limit effort="100" lower="-1.57" upper="1.57" velocity="1"/>
   <dynamics damping="10" friction="0.1"/>
 </joint>
@@ -510,5 +510,5 @@
   <child link="leg_2_link_3__1__1"/>
   <axis xyz="0.126261 -0.010099 -0.991946"/>
-  <limit effort="100" lower="-1.57" upper="1.57" velocity="100"/>
+  <limit effort="100" lower="-1.57" upper="1.57" velocity="1"/>
   <dynamics damping="10" friction="0.1"/>
 </joint>
@@ -518,5 +518,5 @@
   <child link="leg_2_link_2_1"/>
   <axis xyz="-0.079733 -0.996816 0.0"/>
-  <limit effort="100" lower="-1.57" upper="1.57" velocity="100"/>
+  <limit effort="100" lower="-1.57" upper="1.57" velocity="1"/>
   <dynamics damping="10" friction="0.1"/>
 </joint>
@@ -526,5 +526,5 @@
   <child link="leg_2_link_1_1"/>
   <axis xyz="-0.079733 -0.996816 0.0"/>
-  <limit effort="100" lower="-1.57" upper="1.57" velocity="100"/>
+  <limit effort="100" lower="-1.57" upper="1.57" velocity="1"/>
   <dynamics damping="10" friction="0.1"/>
 </joint>
