Commit message: Updated urdf files from aryan/urdf branch

File: hexapod_description/urdf/hexapod.xacro (robot description, xacro)
@@ -4,10 +4,9 @@
 <xacro:include filename="$(find hexapod_description)/urdf/hexapod.trans" />
 <xacro:include filename="$(find hexapod_description)/urdf/hexapod.gazebo" />
-<xacro:include filename="$(find hexapod_control)/ros2_control/ros2_control.xacro" />
 <link name="base_link">
   <inertial>
-    <origin xyz="0.1000352418955988 0.06495559041692857 0.006960329203092366" rpy="0 0 0"/>
+    <origin xyz="0.10909777793044037 0.06468612005136756 0.006889314215312581" rpy="0 0 0"/>
     <mass value="14.09466584247892"/>
-    <inertia ixx="0.167546" iyy="0.075339" izz="0.199615" ixy="-0.012339" iyz="0.003184" ixz="-0.003868"/>
+    <inertia ixx="0.168182" iyy="0.074083" izz="0.200235" ixy="0.006215" iyz="0.001309" ixz="-0.000356"/>
   </inertial>
   <visual>
@@ -27,10 +26,10 @@
 <link name="leg_1_link_2_1">
   <inertial>
-    <origin xyz="-0.020798247907869903 -0.003004122621169035 -0.05840364105605461" rpy="0 0 0"/>
+    <origin xyz="-0.02800590467788834 0.004191461427254562 -0.05523214859518318" rpy="0 0 0"/>
     <mass value="1.012661950148346"/>
-    <inertia ixx="0.001014" iyy="0.001236" izz="0.000891" ixy="-0.000197" iyz="-0.00022" ixz="-0.000489"/>
-  </inertial>
-  <visual>
-    <origin xyz="0.031628 0.00646 -0.021757" rpy="0 0 0"/>
+    <inertia ixx="0.000816" iyy="0.001315" izz="0.00101" ixy="-0.000122" iyz="-8.3e-05" ixz="-0.000522"/>
+  </inertial>
+  <visual>
+    <origin xyz="0.003565 0.030766 -0.036053" rpy="0 0 0"/>
     <geometry>
       <mesh filename="file://$(find hexapod_description)/meshes/leg_1_link_2_1.stl" scale="0.001 0.001 0.001"/>
@@ -39,5 +38,5 @@
   </visual>
   <collision>
-    <origin xyz="0.031628 0.00646 -0.021757" rpy="0 0 0"/>
+    <origin xyz="0.003565 0.030766 -0.036053" rpy="0 0 0"/>
     <geometry>
       <mesh filename="file://$(find hexapod_description)/meshes/leg_1_link_2_1.stl" scale="0.001 0.001 0.001"/>
@@ -47,10 +46,10 @@
 <link name="leg_1_link_3_1">
   <inertial>
-    <origin xyz="-0.05232794213563882 0.015850438170881664 0.012387465467738626" rpy="0 0 0"/>
+    <origin xyz="-0.036766491881322055 0.024823115706118865 0.034277514263341684" rpy="0 0 0"/>
     <mass value="0.22871600239093776"/>
-    <inertia ixx="0.000208" iyy="0.000275" izz="0.000422" ixy="-1e-05" iyz="1.8e-05" ixz="6.7e-05"/>
-  </inertial>
-  <visual>
-    <origin xyz="0.080903 0.053284 0.063455" rpy="0 0 0"/>
+    <inertia ixx="0.000307" iyy="0.000276" izz="0.000321" ixy="-2e-06" iyz="-2e-06" ixz="0.000128"/>
+  </inertial>
+  <visual>
+    <origin xyz="0.071402 0.062467 0.04316" rpy="0 0 0"/>
     <geometry>
       <mesh filename="file://$(find hexapod_description)/meshes/leg_1_link_3_1.stl" scale="0.001 0.001 0.001"/>
@@ -59,5 +58,5 @@
   </visual>
   <collision>
-    <origin xyz="0.080903 0.053284 0.063455" rpy="0 0 0"/>
+    <origin xyz="0.071402 0.062467 0.04316" rpy="0 0 0"/>
     <geometry>
       <mesh filename="file://$(find hexapod_description)/meshes/leg_1_link_3_1.stl" scale="0.001 0.001 0.001"/>
@@ -67,10 +66,10 @@
 <link name="leg_1_link_1_1">
   <inertial>
-    <origin xyz="-0.024118708207036738 0.023198280722906535 -0.02416394528421939" rpy="0 0 0"/>
+    <origin xyz="-0.01779410893760297 0.028725816249512953 -0.02370507712814386" rpy="0 0 0"/>
     <mass value="0.907399585528797"/>
-    <inertia ixx="0.0028" iyy="0.003123" izz="0.0006" ixy="-0.00015" iyz="-0.00034" ixz="-0.000941"/>
-  </inertial>
-  <visual>
-    <origin xyz="0.175395 0.070243 0.035462" rpy="0 0 0"/>
+    <inertia ixx="0.002849" iyy="0.003176" izz="0.000497" ixy="-2.4e-05" iyz="-1.8e-05" ixz="-0.000878"/>
+  </inertial>
+  <visual>
+    <origin xyz="0.144088 0.062627 -0.025519" rpy="0 0 0"/>
     <geometry>
       <mesh filename="file://$(find hexapod_description)/meshes/leg_1_link_1_1.stl" scale="0.001 0.001 0.001"/>
@@ -79,5 +78,5 @@
   </visual>
   <collision>
-    <origin xyz="0.175395 0.070243 0.035462" rpy="0 0 0"/>
+    <origin xyz="0.144088 0.062627 -0.025519" rpy="0 0 0"/>
     <geometry>
       <mesh filename="file://$(find hexapod_description)/meshes/leg_1_link_1_1.stl" scale="0.001 0.001 0.001"/>
@@ -87,10 +86,10 @@
 <link name="leg_3_link_3_1">
   <inertial>
-    <origin xyz="-0.01471532830032863 0.017066498243044487 -0.05783367655412228" rpy="0 0 0"/>
+    <origin xyz="-0.02800203130695705 0.004225621248029748 -0.05523202595087612" rpy="0 0 0"/>
     <mass value="1.0126620006859057"/>
-    <inertia ixx="0.000964" iyy="0.001294" izz="0.000883" ixy="0.000135" iyz="0.000218" ixz="-0.000494"/>
-  </inertial>
-  <visual>
-    <origin xyz="-0.02145 -0.24803 -0.025922" rpy="0 0 0"/>
+    <inertia ixx="0.000815" iyy="0.001315" izz="0.001011" ixy="-0.000122" iyz="-8.2e-05" ixz="-0.000522"/>
+  </inertial>
+  <visual>
+    <origin xyz="-0.00013 -0.229172 -0.040385" rpy="0 0 0"/>
     <geometry>
       <mesh filename="file://$(find hexapod_description)/meshes/leg_3_link_3_1.stl" scale="0.001 0.001 0.001"/>
@@ -99,5 +98,5 @@
   </visual>
   <collision>
-    <origin xyz="-0.02145 -0.24803 -0.025922" rpy="0 0 0"/>
+    <origin xyz="-0.00013 -0.229172 -0.040385" rpy="0 0 0"/>
     <geometry>
       <mesh filename="file://$(find hexapod_description)/meshes/leg_3_link_3_1.stl" scale="0.001 0.001 0.001"/>
@@ -107,10 +106,10 @@
 <link name="leg_3_link_2_1">
   <inertial>
-    <origin xyz="-0.02490321172110873 0.04393892851157011 0.024331856966839732" rpy="0 0 0"/>
+    <origin xyz="-0.038612908125580755 0.024931950622849613 0.03209860064693253" rpy="0 0 0"/>
     <mass value="0.2287158182027981"/>
-    <inertia ixx="0.000248" iyy="0.000272" izz="0.000385" ixy="1.3e-05" iyz="-6.3e-05" ixz="8.6e-05"/>
-  </inertial>
-  <visual>
-    <origin xyz="0.042897 -0.255314 0.061759" rpy="0 0 0"/>
+    <inertia ixx="0.000293" iyy="0.000276" izz="0.000335" ixy="-2e-06" iyz="-3e-06" ixz="0.000126"/>
+  </inertial>
+  <visual>
+    <origin xyz="0.067748 -0.197555 0.038827" rpy="0 0 0"/>
     <geometry>
       <mesh filename="file://$(find hexapod_description)/meshes/leg_3_link_2_1.stl" scale="0.001 0.001 0.001"/>
@@ -119,5 +118,5 @@
   </visual>
   <collision>
-    <origin xyz="0.042897 -0.255314 0.061759" rpy="0 0 0"/>
+    <origin xyz="0.067748 -0.197555 0.038827" rpy="0 0 0"/>
     <geometry>
       <mesh filename="file://$(find hexapod_description)/meshes/leg_3_link_2_1.stl" scale="0.001 0.001 0.001"/>
@@ -127,10 +126,10 @@
 <link name="leg_3_link_1_1">
   <inertial>
-    <origin xyz="0.008717952333481188 0.029799584273488944 -0.027197642277439673" rpy="0 0 0"/>
+    <origin xyz="-0.018585545303067386 0.028750059166235353 -0.023059753696741243" rpy="0 0 0"/>
     <mass value="0.9073986789846695"/>
-    <inertia ixx="0.00313" iyy="0.003181" izz="0.000211" ixy="8e-06" iyz="3.3e-05" ixz="0.000122"/>
-  </inertial>
-  <visual>
-    <origin xyz="0.11862 -0.300684 0.014775" rpy="0 0 0"/>
+    <inertia ixx="0.002786" iyy="0.003177" izz="0.00056" ixy="-2.4e-05" iyz="-1.5e-05" ixz="-0.000957"/>
+  </inertial>
+  <visual>
+    <origin xyz="0.144246 -0.197611 -0.025579" rpy="0 0 0"/>
     <geometry>
       <mesh filename="file://$(find hexapod_description)/meshes/leg_3_link_1_1.stl" scale="0.001 0.001 0.001"/>
@@ -139,5 +138,5 @@
   </visual>
   <collision>
-    <origin xyz="0.11862 -0.300684 0.014775" rpy="0 0 0"/>
+    <origin xyz="0.144246 -0.197611 -0.025579" rpy="0 0 0"/>
     <geometry>
       <mesh filename="file://$(find hexapod_description)/meshes/leg_3_link_1_1.stl" scale="0.001 0.001 0.001"/>
@@ -147,10 +146,10 @@
 <link name="leg_4_link_3_1">
   <inertial>
-    <origin xyz="0.03474109636392422 -0.003845593381223762 -0.051356732674382274" rpy="0 0 0"/>
+    <origin xyz="0.027728117209699726 0.005404822632770333 -0.055329193280975665" rpy="0 0 0"/>
     <mass value="1.0132520108724496"/>
-    <inertia ixx="0.000782" iyy="0.001231" izz="0.001141" ixy="0.000257" iyz="-0.000175" ixz="0.000456"/>
-  </inertial>
-  <visual>
-    <origin xyz="-0.178057 0.050638 -0.048896" rpy="0 0 0"/>
+    <inertia ixx="0.000808" iyy="0.001332" izz="0.001013" ixy="9.8e-05" iyz="-5.7e-05" ixz="0.000528"/>
+  </inertial>
+  <visual>
+    <origin xyz="-0.212413 0.03383 -0.035672" rpy="0 0 0"/>
     <geometry>
       <mesh filename="file://$(find hexapod_description)/meshes/leg_4_link_3_1.stl" scale="0.001 0.001 0.001"/>
@@ -159,5 +158,5 @@
   </visual>
   <collision>
-    <origin xyz="-0.178057 0.050638 -0.048896" rpy="0 0 0"/>
+    <origin xyz="-0.212413 0.03383 -0.035672" rpy="0 0 0"/>
     <geometry>
       <mesh filename="file://$(find hexapod_description)/meshes/leg_4_link_3_1.stl" scale="0.001 0.001 0.001"/>
@@ -167,10 +166,10 @@
 <link name="leg_4_link_2_1">
   <inertial>
-    <origin xyz="-0.010888666203385994 0.026973289808990053 0.04744870332220183" rpy="0 0 0"/>
-    <mass value="0.2286696896275042"/>
-    <inertia ixx="0.00041" iyy="0.000283" izz="0.000211" ixy="-3e-05" iyz="-1.5e-05" ixz="7.4e-05"/>
-  </inertial>
-  <visual>
-    <origin xyz="-0.24657 0.099091 0.02152" rpy="0 0 0"/>
+    <origin xyz="0.032412400507978834 0.026441764186800658 0.03671083209822426" rpy="0 0 0"/>
+    <mass value="0.22866968962750417"/>
+    <inertia ixx="0.000318" iyy="0.000277" izz="0.00031" ixy="5e-06" iyz="-9e-06" ixz="-0.000127"/>
+  </inertial>
+  <visual>
+    <origin xyz="-0.282137 0.062216 0.043908" rpy="0 0 0"/>
     <geometry>
       <mesh filename="file://$(find hexapod_description)/meshes/leg_4_link_2_1.stl" scale="0.001 0.001 0.001"/>
@@ -179,5 +178,5 @@
   </visual>
   <collision>
-    <origin xyz="-0.24657 0.099091 0.02152" rpy="0 0 0"/>
+    <origin xyz="-0.282137 0.062216 0.043908" rpy="0 0 0"/>
     <geometry>
       <mesh filename="file://$(find hexapod_description)/meshes/leg_4_link_2_1.stl" scale="0.001 0.001 0.001"/>
@@ -187,10 +186,10 @@
 <link name="leg_4_link_1_1">
   <inertial>
-    <origin xyz="0.02172755655481845 0.024507117043729182 -0.025464522928266398" rpy="0 0 0"/>
+    <origin xyz="0.014752404637279282 0.029533755446086295 -0.025123760851106607" rpy="0 0 0"/>
     <mass value="0.9074869947367368"/>
-    <inertia ixx="0.003012" iyy="0.003161" izz="0.000357" ixy="6.1e-05" iyz="-0.000166" ixz="0.000626"/>
-  </inertial>
-  <visual>
-    <origin xyz="-0.215846 0.094134 -0.073515" rpy="0 0 0"/>
+    <inertia ixx="0.002963" iyy="0.003182" izz="0.000385" ixy="1.1e-05" iyz="1.5e-05" ixz="0.000701"/>
+  </inertial>
+  <visual>
+    <origin xyz="-0.351763 0.05887 -0.027793" rpy="0 0 0"/>
     <geometry>
       <mesh filename="file://$(find hexapod_description)/meshes/leg_4_link_1_1.stl" scale="0.001 0.001 0.001"/>
@@ -199,5 +198,5 @@
   </visual>
   <collision>
-    <origin xyz="-0.215846 0.094134 -0.073515" rpy="0 0 0"/>
+    <origin xyz="-0.351763 0.05887 -0.027793" rpy="0 0 0"/>
     <geometry>
       <mesh filename="file://$(find hexapod_description)/meshes/leg_4_link_1_1.stl" scale="0.001 0.001 0.001"/>
@@ -207,10 +206,10 @@
 <link name="leg_5_link_3_1">
   <inertial>
-    <origin xyz="0.03431863832487392 -0.006415093388469753 -0.05138466470919113" rpy="0 0 0"/>
+    <origin xyz="0.027727362528310262 0.005406300431649566 -0.05532850946625981" rpy="0 0 0"/>
     <mass value="1.0132520108724496"/>
-    <inertia ixx="0.000831" iyy="0.001185" izz="0.001137" ixy="0.000289" iyz="-0.000215" ixz="0.000441"/>
-  </inertial>
-  <visual>
-    <origin xyz="-0.212362 -0.074971 -0.051984" rpy="0 0 0"/>
+    <inertia ixx="0.000808" iyy="0.001332" izz="0.001013" ixy="9.8e-05" iyz="-5.7e-05" ixz="0.000528"/>
+  </inertial>
+  <visual>
+    <origin xyz="-0.22226 -0.096026 -0.037823" rpy="0 0 0"/>
     <geometry>
       <mesh filename="file://$(find hexapod_description)/meshes/leg_5_link_3_1.stl" scale="0.001 0.001 0.001"/>
@@ -219,5 +218,5 @@
   </visual>
   <collision>
-    <origin xyz="-0.212362 -0.074971 -0.051984" rpy="0 0 0"/>
+    <origin xyz="-0.22226 -0.096026 -0.037823" rpy="0 0 0"/>
     <geometry>
       <mesh filename="file://$(find hexapod_description)/meshes/leg_5_link_3_1.stl" scale="0.001 0.001 0.001"/>
@@ -227,10 +226,10 @@
 <link name="leg_5_llink_2_1">
   <inertial>
-    <origin xyz="0.018771123341369156 0.018755066663032692 0.04938055386133791" rpy="0 0 0"/>
-    <mass value="0.2286696896275042"/>
-    <inertia ixx="0.000416" iyy="0.000289" izz="0.000199" ixy="-4.2e-05" iyz="1.9e-05" ixz="-5.3e-05"/>
-  </inertial>
-  <visual>
-    <origin xyz="-0.276253 -0.021267 0.018967" rpy="0 0 0"/>
+    <origin xyz="0.03396675014480838 0.026560629165649705 0.0358235093671267" rpy="0 0 0"/>
+    <mass value="0.22866968962750417"/>
+    <inertia ixx="0.000318" iyy="0.000277" izz="0.00031" ixy="5e-06" iyz="-9e-06" ixz="-0.000127"/>
+  </inertial>
+  <visual>
+    <origin xyz="-0.291986 -0.067645 0.041757" rpy="0 0 0"/>
     <geometry>
       <mesh filename="file://$(find hexapod_description)/meshes/leg_5_llink_2_1.stl" scale="0.001 0.001 0.001"/>
@@ -239,5 +238,5 @@
   </visual>
   <collision>
-    <origin xyz="-0.276253 -0.021267 0.018967" rpy="0 0 0"/>
+    <origin xyz="-0.291986 -0.067645 0.041757" rpy="0 0 0"/>
     <geometry>
       <mesh filename="file://$(find hexapod_description)/meshes/leg_5_llink_2_1.stl" scale="0.001 0.001 0.001"/>
@@ -247,10 +246,10 @@
 <link name="leg_5_link_1_1">
   <inertial>
-    <origin xyz="0.02550183545753798 0.022180183688185383 -0.02405814830958873" rpy="0 0 0"/>
+    <origin xyz="0.015194262734185393 0.029558917275610747 -0.024828532452773375" rpy="0 0 0"/>
     <mass value="0.9074869947367368"/>
-    <inertia ixx="0.002936" iyy="0.003145" izz="0.000449" ixy="9.4e-05" iyz="-0.00024" ixz="0.000773"/>
-  </inertial>
-  <visual>
-    <origin xyz="-0.297249 -0.011829 -0.078348" rpy="0 0 0"/>
+    <inertia ixx="0.002938" iyy="0.003182" izz="0.00041" ixy="1e-05" iyz="1.9e-05" ixz="0.000746"/>
+  </inertial>
+  <visual>
+    <origin xyz="-0.361611 -0.070996 -0.029944" rpy="0 0 0"/>
     <geometry>
       <mesh filename="file://$(find hexapod_description)/meshes/leg_5_link_1_1.stl" scale="0.001 0.001 0.001"/>
@@ -259,5 +258,5 @@
   </visual>
   <collision>
-    <origin xyz="-0.297249 -0.011829 -0.078348" rpy="0 0 0"/>
+    <origin xyz="-0.361611 -0.070996 -0.029944" rpy="0 0 0"/>
     <geometry>
       <mesh filename="file://$(find hexapod_description)/meshes/leg_5_link_1_1.stl" scale="0.001 0.001 0.001"/>
@@ -267,10 +266,10 @@
 <link name="leg_6_link_3_1">
   <inertial>
-    <origin xyz="0.03478752240465702 -0.0034309973765440926 -0.05135500529375246" rpy="0 0 0"/>
+    <origin xyz="0.027727583128841132 0.005406596018310561 -0.055328604623189385" rpy="0 0 0"/>
     <mass value="1.0132520108724496"/>
-    <inertia ixx="0.000774" iyy="0.001238" izz="0.001142" ixy="0.000252" iyz="-0.000168" ixz="0.000458"/>
-  </inertial>
-  <visual>
-    <origin xyz="-0.231135 -0.203852 -0.053061" rpy="0 0 0"/>
+    <inertia ixx="0.000808" iyy="0.001332" izz="0.001013" ixy="9.8e-05" iyz="-5.7e-05" ixz="0.000528"/>
+  </inertial>
+  <visual>
+    <origin xyz="-0.216108 -0.226108 -0.040003" rpy="0 0 0"/>
     <geometry>
       <mesh filename="file://$(find hexapod_description)/meshes/leg_6_link_3_1.stl" scale="0.001 0.001 0.001"/>
@@ -279,5 +278,5 @@
   </visual>
   <collision>
-    <origin xyz="-0.231135 -0.203852 -0.053061" rpy="0 0 0"/>
+    <origin xyz="-0.216108 -0.226108 -0.040003" rpy="0 0 0"/>
     <geometry>
       <mesh filename="file://$(find hexapod_description)/meshes/leg_6_link_3_1.stl" scale="0.001 0.001 0.001"/>
@@ -287,10 +286,10 @@
 <link name="leg_6_link_2_1">
   <inertial>
-    <origin xyz="0.03849750463385049 0.017157271320907497 0.03696038927730658" rpy="0 0 0"/>
-    <mass value="0.2286696896275042"/>
-    <inertia ixx="0.000325" iyy="0.000278" izz="0.000301" ixy="-8e-06" iyz="2.5e-05" ixz="-0.000125"/>
-  </inertial>
-  <visual>
-    <origin xyz="-0.300343 -0.156279 0.017275" rpy="0 0 0"/>
+    <origin xyz="0.033966970745339664 0.02656092475231095 0.03582341421019737" rpy="0 0 0"/>
+    <mass value="0.22866968962750417"/>
+    <inertia ixx="0.000318" iyy="0.000277" izz="0.00031" ixy="5e-06" iyz="-9e-06" ixz="-0.000127"/>
+  </inertial>
+  <visual>
+    <origin xyz="-0.285834 -0.197727 0.039577" rpy="0 0 0"/>
     <geometry>
       <mesh filename="file://$(find hexapod_description)/meshes/leg_6_link_2_1.stl" scale="0.001 0.001 0.001"/>
@@ -299,5 +298,5 @@
   </visual>
   <collision>
-    <origin xyz="-0.300343 -0.156279 0.017275" rpy="0 0 0"/>
+    <origin xyz="-0.285834 -0.197727 0.039577" rpy="0 0 0"/>
     <geometry>
       <mesh filename="file://$(find hexapod_description)/meshes/leg_6_link_2_1.stl" scale="0.001 0.001 0.001"/>
@@ -307,10 +306,10 @@
 <link name="leg_6_link_1_1">
   <inertial>
-    <origin xyz="0.02586216823859211 0.02382740021676627 -0.022010668931323946" rpy="0 0 0"/>
+    <origin xyz="0.015193483334715818 0.029559212862271284 -0.024828627609704317" rpy="0 0 0"/>
     <mass value="0.9074869947367368"/>
-    <inertia ixx="0.002693" iyy="0.003147" izz="0.00069" ixy="0.00013" iyz="-0.000245" ixz="0.001062"/>
-  </inertial>
-  <visual>
-    <origin xyz="-0.36607 -0.142086 -0.056742" rpy="0 0 0"/>
+    <inertia ixx="0.002938" iyy="0.003182" izz="0.00041" ixy="1e-05" iyz="1.9e-05" ixz="0.000746"/>
+  </inertial>
+  <visual>
+    <origin xyz="-0.35546 -0.201078 -0.032124" rpy="0 0 0"/>
     <geometry>
       <mesh filename="file://$(find hexapod_description)/meshes/leg_6_link_1_1.stl" scale="0.001 0.001 0.001"/>
@@ -319,5 +318,5 @@
   </visual>
   <collision>
-    <origin xyz="-0.36607 -0.142086 -0.056742" rpy="0 0 0"/>
+    <origin xyz="-0.35546 -0.201078 -0.032124" rpy="0 0 0"/>
     <geometry>
       <mesh filename="file://$(find hexapod_description)/meshes/leg_6_link_1_1.stl" scale="0.001 0.001 0.001"/>
@@ -325,21 +324,21 @@
   </collision>
 </link>
-<link name="leg_2_link_3__1__1">
-  <inertial>
-    <origin xyz="-0.0204324626555867 0.004535002979926123 -0.058433485854018384" rpy="0 0 0"/>
+<link name="leg_2_link_3__1">
+  <inertial>
+    <origin xyz="-0.02799670252196973 0.004276094383967741 -0.055230856580649954" rpy="0 0 0"/>
     <mass value="1.0126607300527286"/>
-    <inertia ixx="0.000937" iyy="0.001326" izz="0.000878" ixy="-9.5e-05" iyz="-6.9e-05" ixz="-0.000533"/>
-  </inertial>
-  <visual>
-    <origin xyz="0.012855 -0.122421 -0.022834" rpy="0 0 0"/>
-    <geometry>
-      <mesh filename="file://$(find hexapod_description)/meshes/leg_2_link_3__1__1.stl" scale="0.001 0.001 0.001"/>
-    </geometry>
-    <material name="silver"/>
-  </visual>
-  <collision>
-    <origin xyz="0.012855 -0.122421 -0.022834" rpy="0 0 0"/>
-    <geometry>
-      <mesh filename="file://$(find hexapod_description)/meshes/leg_2_link_3__1__1.stl" scale="0.001 0.001 0.001"/>
+    <inertia ixx="0.000815" iyy="0.001316" izz="0.001011" ixy="-0.000121" iyz="-8.1e-05" ixz="-0.000522"/>
+  </inertial>
+  <visual>
+    <origin xyz="0.009716 -0.099316 -0.038233" rpy="0 0 0"/>
+    <geometry>
+      <mesh filename="file://$(find hexapod_description)/meshes/leg_2_link_3__1.stl" scale="0.001 0.001 0.001"/>
+    </geometry>
+    <material name="silver"/>
+  </visual>
+  <collision>
+    <origin xyz="0.009716 -0.099316 -0.038233" rpy="0 0 0"/>
+    <geometry>
+      <mesh filename="file://$(find hexapod_description)/meshes/leg_2_link_3__1.stl" scale="0.001 0.001 0.001"/>
     </geometry>
   </collision>
@@ -347,10 +346,10 @@
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
File: hexapod_description/urdf/materials.xacro (robot description, xacro)
@@ -2,5 +2,5 @@
 <robot name="hexapod" xmlns:xacro="http://www.ros.org/wiki/xacro" >
 <material name="silver">
-  <color rgba="1.000 0.500 0.700 1.000"/>
+  <color rgba="0.700 0.700 0.700 1.000"/>
 </material>
 </robot>
