Commit message: implemeted very basic IK

File: hexapod_description/urdf/hexapod.xacro (robot description, xacro)
@@ -391,5 +391,5 @@
   <axis xyz="-0.001529 0.016683 -0.99986"/>
   <limit effort="100" lower="-1.57" upper="0.785" velocity="100"/>
-  <dynamics damping="10" friction="0.1"/>
+  <dynamics damping="10" friction="0.5"/>
 </joint>
 <joint name="Leg_1_tibia" type="revolute">
@@ -399,5 +399,5 @@
   <axis xyz="-0.013531 -0.99977 -0.016661"/>
   <limit effort="100" lower="-1.57" upper="1.57" velocity="100"/>
-  <dynamics damping="10" friction="0.1"/>
+  <dynamics damping="10" friction="0.5"/>
 </joint>
 <joint name="Leg_1_femur" type="revolute">
@@ -407,5 +407,5 @@
   <axis xyz="-0.013531 -0.99977 -0.016661"/>
   <limit effort="100" lower="-1.57" upper="1.57" velocity="100"/>
-  <dynamics damping="10" friction="0.1"/>
+  <dynamics damping="10" friction="0.5"/>
 </joint>
 <joint name="Leg_3_coxa" type="revolute">
@@ -415,5 +415,5 @@
   <axis xyz="-0.001529 0.016683 -0.99986"/>
   <limit effort="100" lower="-0.785" upper="1.57" velocity="100"/>
-  <dynamics damping="10" friction="0.1"/>
+  <dynamics damping="10" friction="0.5"/>
 </joint>
 <joint name="Leg_3_tibia" type="revolute">
@@ -423,5 +423,5 @@
   <axis xyz="-0.014767 -0.999752 -0.016659"/>
   <limit effort="100" lower="-1.57" upper="1.57" velocity="100"/>
-  <dynamics damping="10" friction="0.1"/>
+  <dynamics damping="10" friction="0.5"/>
 </joint>
 <joint name="Leg_3_femur" type="revolute">
@@ -431,5 +431,5 @@
   <axis xyz="-0.014767 -0.999752 -0.016659"/>
   <limit effort="100" lower="-1.57" upper="1.57" velocity="100"/>
-  <dynamics damping="10" friction="0.1"/>
+  <dynamics damping="10" friction="0.5"/>
 </joint>
 <joint name="Leg_4_coxa" type="revolute">
@@ -439,5 +439,5 @@
   <axis xyz="-0.001529 0.016683 -0.99986"/>
   <limit effort="100" lower="-0.785" upper="1.57" velocity="100"/>
-  <dynamics damping="10" friction="0.1"/>
+  <dynamics damping="10" friction="0.5"/>
 </joint>
 <joint name="Leg_5_coxa" type="revolute">
@@ -447,5 +447,5 @@
   <axis xyz="-0.001529 0.016683 -0.99986"/>
   <limit effort="100" lower="-0.785" upper="0.785" velocity="100"/>
-  <dynamics damping="10" friction="0.1"/>
+  <dynamics damping="10" friction="0.5"/>
 </joint>
 <joint name="Leg_5_tibia" type="revolute">
@@ -455,5 +455,5 @@
   <axis xyz="0.065266 -0.997727 -0.016747"/>
   <limit effort="100" lower="-1.57" upper="1.57" velocity="100"/>
-  <dynamics damping="10" friction="0.1"/>
+  <dynamics damping="10" friction="0.5"/>
 </joint>
 <joint name="Leg_5_femur" type="revolute">
@@ -463,5 +463,5 @@
   <axis xyz="-0.065266 0.997727 0.016747"/>
   <limit effort="100" lower="-1.57" upper="1.57" velocity="100"/>
-  <dynamics damping="10" friction="0.1"/>
+  <dynamics damping="10" friction="0.5"/>
 </joint>
 <joint name="Leg_6_coxa" type="revolute">
@@ -471,5 +471,5 @@
   <axis xyz="-0.001529 0.016683 -0.99986"/>
   <limit effort="100" lower="-1.57" upper="0.785" velocity="100"/>
-  <dynamics damping="10" friction="0.1"/>
+  <dynamics damping="10" friction="0.5"/>
 </joint>
 <joint name="Leg_6_tibia" type="revolute">
@@ -479,5 +479,5 @@
   <axis xyz="0.065266 -0.997727 -0.016747"/>
   <limit effort="100" lower="-1.57" upper="1.57" velocity="100"/>
-  <dynamics damping="10" friction="0.1"/>
+  <dynamics damping="10" friction="0.5"/>
 </joint>
 <joint name="Leg_6_femur" type="revolute">
@@ -487,5 +487,5 @@
   <axis xyz="-0.065266 0.997727 0.016747"/>
   <limit effort="100" lower="-1.57" upper="1.57" velocity="100"/>
-  <dynamics damping="10" friction="0.1"/>
+  <dynamics damping="10" friction="0.5"/>
 </joint>
 <joint name="Leg_2_coxa" type="revolute">
@@ -495,5 +495,5 @@
   <axis xyz="-0.001529 0.016683 -0.99986"/>
   <limit effort="100" lower="-0.785" upper="0.785" velocity="100"/>
-  <dynamics damping="10" friction="0.1"/>
+  <dynamics damping="10" friction="0.5"/>
 </joint>
 <joint name="Leg_2_tibia" type="revolute">
@@ -503,5 +503,5 @@
   <axis xyz="-0.016551 -0.999724 -0.016656"/>
   <limit effort="100" lower="-1.57" upper="1.57" velocity="100"/>
-  <dynamics damping="10" friction="0.1"/>
+  <dynamics damping="10" friction="0.5"/>
 </joint>
 <joint name="Leg_2_femur" type="revolute">
@@ -511,5 +511,5 @@
   <axis xyz="-0.016551 -0.999724 -0.016656"/>
   <limit effort="100" lower="-1.57" upper="1.57" velocity="100"/>
-  <dynamics damping="10" friction="0.1"/>
+  <dynamics damping="10" friction="0.5"/>
 </joint>
 <joint name="Leg_4_tibia" type="revolute">
@@ -519,5 +519,5 @@
   <axis xyz="0.041169 -0.999012 -0.016732"/>
   <limit effort="100" lower="-1.57" upper="1.57" velocity="100"/>
-  <dynamics damping="10" friction="0.1"/>
+  <dynamics damping="10" friction="0.5"/>
 </joint>
 <joint name="Leg_4_femur" type="revolute">
@@ -527,5 +527,5 @@
   <axis xyz="-0.041169 0.999012 0.016732"/>
   <limit effort="100" lower="-1.57" upper="1.57" velocity="100"/>
-  <dynamics damping="10" friction="0.1"/>
+  <dynamics damping="10" friction="0.5"/>
 </joint>
 </robot>

Commit message: need to fix IK

File: hexapod_description/urdf/hexapod.xacro (robot description, xacro)
@@ -36,5 +36,5 @@
       <mesh filename="file://$(find hexapod_description)/meshes/leg_1_link_2_1.stl" scale="0.001 0.001 0.001"/>
     </geometry>
-    <material name="silver"/>
+    <material name="gold"/>
   </visual>
   <collision>
@@ -96,5 +96,5 @@
       <mesh filename="file://$(find hexapod_description)/meshes/leg_3_link_3_1.stl" scale="0.001 0.001 0.001"/>
     </geometry>
-    <material name="silver"/>
+    <material name="gold"/>
   </visual>
   <collision>
@@ -156,5 +156,5 @@
       <mesh filename="file://$(find hexapod_description)/meshes/leg_4_link_3_1.stl" scale="0.001 0.001 0.001"/>
     </geometry>
-    <material name="silver"/>
+    <material name="gold"/>
   </visual>
   <collision>
@@ -176,5 +176,5 @@
       <mesh filename="file://$(find hexapod_description)/meshes/leg_5_link_3_1.stl" scale="0.001 0.001 0.001"/>
     </geometry>
-    <material name="silver"/>
+    <material name="gold"/>
   </visual>
   <collision>
@@ -236,5 +236,5 @@
       <mesh filename="file://$(find hexapod_description)/meshes/leg_6_link_3_1.stl" scale="0.001 0.001 0.001"/>
     </geometry>
-    <material name="silver"/>
+    <material name="gold"/>
   </visual>
   <collision>
@@ -296,5 +296,5 @@
       <mesh filename="file://$(find hexapod_description)/meshes/leg_2_link_3__1.stl" scale="0.001 0.001 0.001"/>
     </geometry>
-    <material name="silver"/>
+    <material name="gold"/>
   </visual>
   <collision>

File: hexapod_description/urdf/materials.xacro (robot description, xacro)
@@ -4,3 +4,6 @@
   <color rgba="0.100 0.100 0.100 1.000"/>
 </material>
+<material name="gold">
+  <color rgba="0.90 0.90 0.00 1.000"/>
+</material>
 </robot>

Commit message: minor changes in IK implementation

File: hexapod_description/urdf/hexapod.xacro (robot description, xacro)
@@ -393,5 +393,5 @@
   <dynamics damping="10" friction="0.5"/>
 </joint>
-<joint name="Leg_1_tibia" type="revolute">
+<joint name="Leg_1_femur" type="revolute">
   <origin xyz="-0.067837 -0.031701 -0.079213" rpy="0 0 0"/>
   <parent link="leg_1_link_2_1"/>
@@ -401,5 +401,5 @@
   <dynamics damping="10" friction="0.5"/>
 </joint>
-<joint name="Leg_1_femur" type="revolute">
+<joint name="Leg_1_tibia" type="revolute">
   <origin xyz="-0.072686 -0.00016 0.068679" rpy="0 0 0"/>
   <parent link="leg_1_link_3_1"/>
@@ -417,5 +417,5 @@
   <dynamics damping="10" friction="0.5"/>
 </joint>
-<joint name="Leg_3_tibia" type="revolute">
+<joint name="Leg_3_femur" type="revolute">
   <origin xyz="-0.067878 -0.031617 -0.079212" rpy="0 0 0"/>
   <parent link="leg_3_link_3_1"/>
@@ -425,5 +425,5 @@
   <dynamics damping="10" friction="0.5"/>
 </joint>
-<joint name="Leg_3_femur" type="revolute">
+<joint name="Leg_3_tibia" type="revolute">
   <origin xyz="-0.076498 5.6e-05 0.064406" rpy="0 0 0"/>
   <parent link="leg_3_link_2_1"/>
@@ -449,5 +449,5 @@
   <dynamics damping="10" friction="0.5"/>
 </joint>
-<joint name="Leg_5_tibia" type="revolute">
+<joint name="Leg_5_femur" type="revolute">
   <origin xyz="0.069726 -0.028381 -0.07958" rpy="0 0 0"/>
   <parent link="leg_5_link_3_1"/>
@@ -457,5 +457,5 @@
   <dynamics damping="10" friction="0.5"/>
 </joint>
-<joint name="Leg_5_femur" type="revolute">
+<joint name="Leg_5_tibia" type="revolute">
   <origin xyz="0.069625 0.003351 0.071701" rpy="0 0 0"/>
   <parent link="leg_5_llink_2_1"/>
@@ -473,5 +473,5 @@
   <dynamics damping="10" friction="0.5"/>
 </joint>
-<joint name="Leg_6_tibia" type="revolute">
+<joint name="Leg_6_femur" type="revolute">
   <origin xyz="0.069726 -0.028381 -0.07958" rpy="0 0 0"/>
   <parent link="leg_6_link_3_1"/>
@@ -481,5 +481,5 @@
   <dynamics damping="10" friction="0.5"/>
 </joint>
-<joint name="Leg_6_femur" type="revolute">
+<joint name="Leg_6_tibia" type="revolute">
   <origin xyz="0.069626 0.003351 0.071701" rpy="0 0 0"/>
   <parent link="leg_6_link_2_1"/>
@@ -497,5 +497,5 @@
   <dynamics damping="10" friction="0.5"/>
 </joint>
-<joint name="Leg_2_tibia" type="revolute">
+<joint name="Leg_2_femur" type="revolute">
   <origin xyz="-0.067937 -0.031496 -0.079209" rpy="0 0 0"/>
   <parent link="leg_2_link_3__1"/>
@@ -505,5 +505,5 @@
   <dynamics damping="10" friction="0.5"/>
 </joint>
-<joint name="Leg_2_femur" type="revolute">
+<joint name="Leg_2_tibia" type="revolute">
   <origin xyz="-0.072405 5e-05 0.068975" rpy="0 0 0"/>
   <parent link="leg_2_link_2_1"/>
@@ -513,5 +513,5 @@
   <dynamics damping="10" friction="0.5"/>
 </joint>
-<joint name="Leg_4_tibia" type="revolute">
+<joint name="Leg_4_femur" type="revolute">
   <origin xyz="0.068989 -0.030057 -0.079607" rpy="0 0 0"/>
   <parent link="leg_4_link_3_1"/>
@@ -521,5 +521,5 @@
   <dynamics damping="10" friction="0.5"/>
 </joint>
-<joint name="Leg_4_femur" type="revolute">
+<joint name="Leg_4_tibia" type="revolute">
   <origin xyz="0.069715 0.001672 0.071673" rpy="0 0 0"/>
   <parent link="leg_4_link_2_1"/>

Commit message: added colours to hexapod

File: hexapod_description/urdf/hexapod.xacro (robot description, xacro)
@@ -36,5 +36,5 @@
       <mesh filename="file://$(find hexapod_description)/meshes/leg_1_coxa_1.stl" scale="0.001 0.001 0.001"/>
     </geometry>
-    <material name="silver"/>
+    <material name="gold"/>
   </visual>
   <collision>
@@ -96,5 +96,5 @@
       <mesh filename="file://$(find hexapod_description)/meshes/leg_3_coxa_1.stl" scale="0.001 0.001 0.001"/>
     </geometry>
-    <material name="silver"/>
+    <material name="gold"/>
   </visual>
   <collision>
@@ -156,5 +156,5 @@
       <mesh filename="file://$(find hexapod_description)/meshes/leg_4_coxa_1.stl" scale="0.001 0.001 0.001"/>
     </geometry>
-    <material name="silver"/>
+    <material name="gold"/>
   </visual>
   <collision>
@@ -176,5 +176,5 @@
       <mesh filename="file://$(find hexapod_description)/meshes/leg_5_coxa_1.stl" scale="0.001 0.001 0.001"/>
     </geometry>
-    <material name="silver"/>
+    <material name="gold"/>
   </visual>
   <collision>
@@ -236,5 +236,5 @@
       <mesh filename="file://$(find hexapod_description)/meshes/leg_6_coxa_1.stl" scale="0.001 0.001 0.001"/>
     </geometry>
-    <material name="silver"/>
+    <material name="gold"/>
   </visual>
   <collision>
@@ -296,5 +296,5 @@
       <mesh filename="file://$(find hexapod_description)/meshes/leg_2_coxa_1.stl" scale="0.001 0.001 0.001"/>
     </geometry>
-    <material name="silver"/>
+    <material name="gold"/>
   </visual>
   <collision>

File: hexapod_description/urdf/materials.xacro (robot description, xacro)
@@ -2,5 +2,8 @@
 <robot name="hexapod" xmlns:xacro="http://www.ros.org/wiki/xacro" >
 <material name="silver">
-  <color rgba="0.700 0.700 0.700 1.000"/>
+  <color rgba="0.100 0.100 0.100 1.000"/>
+</material>
+<material name="gold">
+  <color rgba="0.90 0.90 0.00 1.000"/>
 </material>
 </robot>
